File: DriveBoard_Hardware/DriveBoard_Hardware.sch (KiCad schematic (older format))
At the start: 23 parts

Commit message: Cleaned up, organized, and labeled schematic components
Parts:
- gave numbers to parts that had none: 12
- renumbered C7 to C1, C5 to C10, C1 to C3, C2 to C4, C3 to C7, C6 to C8, C4 to C9
Other:
- note added: "Motor Control Serial Lines"
- note added: "Power Filtration System"
- note added: "Serial Connector I/O"
- note added: "Tiva-IC Serial Lines"

Commit message: Assigned packages and created layout
Parts:
- C1, C10, C11, C12, C2, C3, C4, C5, C6, C7, C8, C9: footprint (none) -> Capacitor_SMD:C_0603_1608Metric_Pad1.05x0.95mm_HandSolder
- Conn1: footprint (none) -> MRDT_Connectors:Anderson_2_Horisontal_Side_by_Side
- Conn2, Conn3, Conn4: footprint (none) -> MRDT_Connectors:MOLEX_SL_05_Horizontal
- U1, U2: footprint (none) -> Package_SO:SOIC-16_3.9x9.9mm_P1.27mm
- U3: footprint (none) -> MRDT_Devices:OKI_Horizontal
- U4: footprint (none) -> MRDT_Shields:TM4C129E_Launchpad_X7_Bottom_SMD
Connections:
- net labels removed: Motor1,2, Motor3,4, Motor5,6
Other:
- note added: "Connectors"
- note added: "Level Shifters"
- note added: "Motor 1,2"
- note added: "Motor 3,4"
- note added: "Motor 5,6"
- note added: "Power Filtering"
- note added: "Serial 3"
- note added: "Serial 4"
- note added: "Serial 6"
- note added: "Tiva Headers"
- note removed: "Motor Control Serial Lines"
- note removed: "Power Filtration System"
- note removed: "Serial Connector I/O"
- note removed: "Tiva-IC Serial Lines"
Changed lines of the file:
@@
 F 0 "U3" H 4250 2050 60  0001 C CNN
 F 1 "OKI" H 4400 2381 60  0000 C CNN
-F 2 "" H 4000 2000 60  0001 C CNN
+F 2 "MRDT_Devices:OKI_Horizontal" H 4000 2000 60  0001 C CNN
 F 3 "" H 4000 2000 60  0001 C CNN
 	1    4200 2100
@@
 F 0 "Conn1" H 3256 2681 60  0000 C CNN
 F 1 "AndersonPP" H 3256 2681 60  0001 C CNN
-F 2 "" H 2900 1850 60  0001 C CNN
+F 2 "MRDT_Connectors:Anderson_2_Horisontal_Side_by_Side" H 2900 1850 60  0001 C CNN
 F 3 "" H 2900 1850 60  0001 C CNN
 	1    3050 2400
@@
 F 0 "Conn1" H 3256 2381 60  0000 C CNN
 F 1 "AndersonPP" H 3256 2381 60  0001 C CNN
-F 2 "" H 2900 1550 60  0001 C CNN
+F 2 "MRDT_Connectors:Anderson_2_Horisontal_Side_by_Side" H 2900 1550 60  0001 C CNN
 F 3 "" H 2900 1550 60  0001 C CNN
 	2    3050 2100
@@
 F 0 "C7" H 3915 2196 50  0000 L CNN
 F 1 "10uF" H 3915 2105 50  0000 L CNN
-F 2 "" H 3838 2000 50  0001 C CNN
+F 2 "Capacitor_SMD:C_0603_1608Metric_Pad1.05x0.95mm_HandSolder" H 3838 2000 50  0001 C CNN
 F 3 "~" H 3800 2150 50  0001 C CNN
 	1    3800 2150
@@
 F 0 "C8" H 5115 2196 50  0000 L CNN
 F 1 "10uF" H 5115 2105 50  0000 L CNN
-F 2 "" H 5038 2000 50  0001 C CNN
+F 2 "Capacitor_SMD:C_0603_1608Metric_Pad1.05x0.95mm_HandSolder" H 5038 2000 50  0001 C CNN
 F 3 "~" H 5000 2150 50  0001 C CNN
 	1    5000 2150
@@
 F 0 "U1" H 4300 6087 60  0000 C CNN
 F 1 "MAX_3232" H 4300 5981 60  0000 C CNN
-F 2 "" H 3950 4150 60  0001 C CNN
+F 2 "Package_SO:SOIC-16_3.9x9.9mm_P1.27mm" H 3950 4150 60  0001 C CNN
 F 3 "" H 3950 4150 60  0001 C CNN
 	1    3950 4750
@@
 F 0 "C9" H 5365 3846 50  0000 L CNN
 F 1 ".1uF" H 5365 3755 50  0000 L CNN
-F 2 "" H 5288 3650 50  0001 C CNN
+F 2 "Capacitor_SMD:C_0603_1608Metric_Pad1.05x0.95mm_HandSolder" H 5288 3650 50  0001 C CNN
 F 3 "~" H 5250 3800 50  0001 C CNN
 	1    5250 3800
@@
 F 0 "C10" H 5365 4196 50  0000 L CNN
 F 1 ".1uF" H 5365 4105 50  0000 L CNN
-F 2 "" H 5288 4000 50  0001 C CNN
+F 2 "Capacitor_SMD:C_0603_1608Metric_Pad1.05x0.95mm_HandSolder" H 5288 4000 50  0001 C CNN
 F 3 "~" H 5250 4150 50  0001 C CNN
 	1    5250 4150
@@
 F 0 "C3" V 3500 4000 50  0000 C CNN
 F 1 ".1uF" V 3500 4250 50  0000 C CNN
-F 2 "" H 3488 3950 50  0001 C CNN
+F 2 "Capacitor_SMD:C_0603_1608Metric_Pad1.05x0.95mm_HandSolder" H 3488 3950 50  0001 C CNN
 F 3 "~" H 3450 4100 50  0001 C CNN
 	1    3450 4100
@@
 F 0 "C4" V 3400 4100 50  0000 C CNN
 F 1 ".1uF" V 3400 4350 50  0000 C CNN
-F 2 "" H 3488 4050 50  0001 C CNN
+F 2 "Capacitor_SMD:C_0603_1608Metric_Pad1.05x0.95mm_HandSolder" H 3488 4050 50  0001 C CNN
 F 3 "~" H 3450 4200 50  0001 C CNN
 	1    3450 4200
@@
 F 0 "Conn2" H 7377 1808 60  0000 L CNN
 F 1 "Molex_SL_05" H 7377 1702 60  0000 L CNN
-F 2 "" H 7250 1500 60  0001 C CNN
+F 2 "MRDT_Connectors:MOLEX_SL_05_Horizontal" H 7250 1500 60  0001 C CNN
 F 3 "" H 7250 1500 60  0001 C CNN
 	1    7250 1500
@@
 F 0 "Conn3" H 7377 2508 60  0000 L CNN
 F 1 "Molex_SL_05" H 7377 2402 60  0000 L CNN
-F 2 "" H 7250 2200 60  0001 C CNN
+F 2 "MRDT_Connectors:MOLEX_SL_05_Horizontal" H 7250 2200 60  0001 C CNN
 F 3 "" H 7250 2200 60  0001 C CNN
 	1    7250 2200
@@
 F 0 "Conn4" H 7377 3158 60  0000 L CNN
 F 1 "Molex_SL_05" H 7377 3052 60  0000 L CNN
-F 2 "" H 7250 2850 60  0001 C CNN
+F 2 "MRDT_Connectors:MOLEX_SL_05_Horizontal" H 7250 2850 60  0001 C CNN
 F 3 "" H 7250 2850 60  0001 C CNN
 	1    7250 2850
@@
 F 0 "C1" H 3465 3796 50  0000 L CNN
 F 1 ".1uF" H 3465 3705 50  0000 L CNN
-F 2 "" H 3388 3600 50  0001 C CNN
+F 2 "Capacitor_SMD:C_0603_1608Metric_Pad1.05x0.95mm_HandSolder" H 3388 3600 50  0001 C CNN
 F 3 "~" H 3350 3750 50  0001 C CNN
 	1    3350 3750
@@
 Wire Wire Line
 	6500 2600 6500 2650
-Text Label 7350 1400 1    50   ~ 0
-Motor1,2
-Text Label 7350 2100 1    50   ~ 0
-Motor3,4
-Text Label 7350 2750 1    50   ~ 0
-Motor5,6
 $Comp
 L MRDT_ICs:MAX_3232 U2
@@
 F 0 "U2" H 4300 7587 60  0000 C CNN
 F 1 "MAX_3232" H 4300 7481 60  0000 C CNN
-F 2 "" H 3950 5650 60  0001 C CNN
+F 2 "Package_SO:SOIC-16_3.9x9.9mm_P1.27mm" H 3950 5650 60  0001 C CNN
 F 3 "" H 3950 5650 60  0001 C CNN
 	1    3950 6250
@@
 F 0 "C11" H 5365 5346 50  0000 L CNN
 F 1 ".1uF" H 5365 5255 50  0000 L CNN
-F 2 "" H 5288 5150 50  0001 C CNN
+F 2 "Capacitor_SMD:C_0603_1608Metric_Pad1.05x0.95mm_HandSolder" H 5288 5150 50  0001 C CNN
 F 3 "~" H 5250 5300 50  0001 C CNN
 	1    5250 5300
@@
 F 0 "C12" H 5365 5696 50  0000 L CNN
 F 1 ".1uF" H 5365 5605 50  0000 L CNN
-F 2 "" H 5288 5500 50  0001 C CNN
+F 2 "Capacitor_SMD:C_0603_1608Metric_Pad1.05x0.95mm_HandSolder" H 5288 5500 50  0001 C CNN
 F 3 "~" H 5250 5650 50  0001 C CNN
 	1    5250 5650
@@
 F 0 "C5" V 3500 5500 50  0000 C CNN
 F 1 ".1uF" V 3500 5750 50  0000 C CNN
-F 2 "" H 3488 5450 50  0001 C CNN
+F 2 "Capacitor_SMD:C_0603_1608Metric_Pad1.05x0.95mm_HandSolder" H 3488 5450 50  0001 C CNN
 F 3 "~" H 3450 5600 50  0001 C CNN
 	1    3450 5600
@@
 F 0 "C6" V 3400 5600 50  0000 C CNN
 F 1 ".1uF" V 3400 5850 50  0000 C CNN
-F 2 "" H 3488 5550 50  0001 C CNN
+F 2 "Capacitor_SMD:C_0603_1608Metric_Pad1.05x0.95mm_HandSolder" H 3488 5550 50  0001 C CNN
 F 3 "~" H 3450 5700 50  0001 C CNN
 	1    3450 5700
@@
 F 0 "C2" H 3465 5296 50  0000 L CNN
 F 1 ".1uF" H 3465 5205 50  0000 L CNN
-F 2 "" H 3388 5100 50  0001 C CNN
+F 2 "Capacitor_SMD:C_0603_1608Metric_Pad1.05x0.95mm_HandSolder" H 3388 5100 50  0001 C CNN
 F 3 "~" H 3350 5250 50  0001 C CNN
 	1    3350 5250
@@
 F 0 "U4" H 7100 4750 60  0000 L CNN
 F 1 "TM4C129E_Launchpad" H 6850 6500 60  0001 L CNN
-F 2 "" H 7050 4850 60  0001 C CNN
+F 2 "MRDT_Shields:TM4C129E_Launchpad_X7_Bottom_SMD" H 7050 4850 60  0001 C CNN
 F 3 "" H 7050 4850 60  0001 C CNN
 	5    7050 4850
@@
 F 0 "U4" H 7700 4750 60  0000 C CNN
 F 1 "TM4C129E_Launchpad" H 7750 6050 60  0000 C CNN
-F 2 "" H 7550 4850 60  0001 C CNN
+F 2 "MRDT_Shields:TM4C129E_Launchpad_X7_Bottom_SMD" H 7550 4850 60  0001 C CNN
 F 3 "" H 7550 4850 60  0001 C CNN
 	6    7550 4850
@@
 F 0 "U4" H 7050 6050 60  0000 L CNN
 F 1 "TM4C129E_Launchpad" H 7355 6642 60  0001 L CNN
-F 2 "" H 7050 6150 60  0001 C CNN
+F 2 "MRDT_Shields:TM4C129E_Launchpad_X7_Bottom_SMD" H 7050 6150 60  0001 C CNN
 F 3 "" H 7050 6150 60  0001 C CNN
 	7    7050 6150
@@
 F 0 "U4" H 7650 6050 60  0000 C CNN
 F 1 "TM4C129E_Launchpad" H 7750 7350 60  0001 C CNN
-F 2 "" H 7550 6150 60  0001 C CNN
+F 2 "MRDT_Shields:TM4C129E_Launchpad_X7_Bottom_SMD" H 7550 6150 60  0001 C CNN
 F 3 "" H 7550 6150 60  0001 C CNN
 	8    7550 6150
@@
 Wire Notes Line
 	8750 3050 2650 3050
-Text Notes 3400 1250 0    98   ~ 20
-Power Filtration System
-Text Notes 6450 850  0    98   ~ 20
-Serial Connector I/O
-Text Notes 3300 3250 0    98   ~ 20
-Motor Control Serial Lines
-Text Notes 6300 3300 0    98   ~ 20
-Tiva-IC Serial Lines
+Text Notes 6900 850  0    98   ~ 20
+Connectors
+Text Notes 6850 3350 0    98   ~ 20
+Tiva Headers
+Text Notes 3800 1250 0    98   ~ 20
+Power Filtering
+Text Notes 3850 3250 0    98   ~ 20
+Level Shifters
+Text Notes 7350 1450 1    59   ~ 12
+Motor 1,2
+Text Notes 7350 2150 1    59   ~ 12
+Motor 3,4
+Text Notes 7350 2800 1    59   ~ 12
+Motor 5,6
+Text Notes 8100 4250 0    59   ~ 0
+Serial 4
+Text Notes 7900 4650 0    59   ~ 0
+Serial 3
+Text Notes 6300 4050 0    59   ~ 0
+Serial 6
 $EndSCHEMATC

Commit message: Added PDR text files and made a few changes
Connections:
- net labels added: +12V
Changed lines of the file:
@@
 Text Notes 6300 4050 0    59   ~ 0
 Serial 6
+Text Label 3550 2000 0    50   ~ 0
++12V
 $EndSCHEMATC

Commit message: Revised molex pins and created pin layout and connections txt files
Connections:
- wire segments 86 -> 78
Changed lines of the file:
@@
 L power:GND #PWR07
 U 1 1 5BC72384
-P 6450 1250
-F 0 "#PWR07" H 6450 1000 50  0001 C CNN
-F 1 "GND" H 6455 1077 50  0000 C CNN
-F 2 "" H 6450 1250 50  0001 C CNN
-F 3 "" H 6450 1250 50  0001 C CNN
-	1    6450 1250
+P 6950 1450
+F 0 "#PWR07" H 6950 1200 50  0001 C CNN
+F 1 "GND" H 6955 1277 50  0000 C CNN
+F 2 "" H 6950 1450 50  0001 C CNN
+F 3 "" H 6950 1450 50  0001 C CNN
+	1    6950 1450
 	1    0    0    -1
 $EndComp
@@
 L power:GND #PWR08
 U 1 1 5BC723BE
-P 6500 2000
-F 0 "#PWR08" H 6500 1750 50  0001 C CNN
-F 1 "GND" H 6505 1827 50  0000 C CNN
-F 2 "" H 6500 2000 50  0001 C CNN
-F 3 "" H 6500 2000 50  0001 C CNN
-	1    6500 2000
+P 6950 2150
+F 0 "#PWR08" H 6950 1900 50  0001 C CNN
+F 1 "GND" H 6955 1977 50  0000 C CNN
+F 2 "" H 6950 2150 50  0001 C CNN
+F 3 "" H 6950 2150 50  0001 C CNN
+	1    6950 2150
 	1    0    0    -1
 $EndComp
@@
 L power:GND #PWR09
 U 1 1 5BC72410
-P 6500 2650
-F 0 "#PWR09" H 6500 2400 50  0001 C CNN
-F 1 "GND" H 6505 2477 50  0000 C CNN
-F 2 "" H 6500 2650 50  0001 C CNN
-F 3 "" H 6500 2650 50  0001 C CNN
-	1    6500 2650
+P 6950 2800
+F 0 "#PWR09" H 6950 2550 50  0001 C CNN
+F 1 "GND" H 6955 2627 50  0000 C CNN
+F 2 "" H 6950 2800 50  0001 C CNN
+F 3 "" H 6950 2800 50  0001 C CNN
+	1    6950 2800
 	1    0    0    -1
 $EndComp
-Text GLabel 6950 1450 0    50   Output ~ 0
+Text GLabel 7050 1050 0    50   Output ~ 0
 RX_1_SL
 Wire Wire Line
 	7050 1450 6950 1450
-Text GLabel 6950 1350 0    50   Input ~ 0
+Text GLabel 7050 1150 0    50   Input ~ 0
 TX_1_SL
-Wire Wire Line
-	7050 1350 6950 1350
-Wire Wire Line
-	7050 1250 6450 1250
-Text GLabel 6950 2050 0    50   Input ~ 0
+Text GLabel 7050 1850 0    50   Input ~ 0
 TX_2_SL
-Wire Wire Line
-	7050 2050 6950 2050
 $Comp
 L Device:C C1
@@
 Wire Wire Line
 	3600 3600 3600 3700
-Text GLabel 6950 2150 0    50   Output ~ 0
+Text GLabel 7050 1750 0    50   Output ~ 0
 RX_2_SL
 Wire Wire Line
 	7050 2150 6950 2150
-Wire Wire Line
-	7050 1950 6500 1950
-Wire Wire Line
-	6500 1950 6500 2000
-Text GLabel 6950 2700 0    50   Input ~ 0
+Text GLabel 7050 2500 0    50   Input ~ 0
 TX_3_SL
-Text GLabel 6950 2800 0    50   Output ~ 0
+Text GLabel 7050 2400 0    50   Output ~ 0
 RX_3_SL
 Wire Wire Line
-	7050 2700 6950 2700
-Wire Wire Line
 	7050 2800 6950 2800
-Wire Wire Line
-	7050 2600 6500 2600
-Wire Wire Line
-	6500 2600 6500 2650
 $Comp
 L MRDT_ICs:MAX_3232 U2

Commit message: Placed components that need to replace oki
Parts:
- added D?: LED, symbol Device:LED
- added R?: 100, symbol Device:R_Small
- added U?: AP1059, symbol MRDT_ICs:AP1059
Changed lines of the file:
@@
 Text Label 3550 2000 0    50   ~ 0
 +12V
+$Comp
+L MRDT_ICs:AP1059 U?
+U 1 1 5BE8A9F0
+P 9450 2300
+F 0 "U?" H 9675 2897 60  0000 C CNN
+F 1 "AP1059" H 9675 2791 60  0000 C CNN
+F 2 "" H 9200 2200 60  0001 C CNN
+F 3 "" H 9200 2200 60  0001 C CNN
+	1    9450 2300
+	1    0    0    -1
+$EndComp
+$Comp
+L Device:LED D?
+U 1 1 5BE8AD8F
+P 5650 2100
+F 0 "D?" V 5688 1983 50  0000 R CNN
+F 1 "LED" V 5597 1983 50  0000 R CNN
+F 2 "" H 5650 2100 50  0001 C CNN
+F 3 "~" H 5650 2100 50  0001 C CNN
+	1    5650 2100
+	0    -1   -1   0
+$EndComp
+$Comp
+L Device:R_Small R?
+U 1 1 5BE8AEA0
+P 5650 1800
+F 0 "R?" H 5709 1846 50  0000 L CNN
+F 1 "100" H 5709 1755 50  0000 L CNN
+F 2 "" H 5650 1800 50  0001 C CNN
+F 3 "~" H 5650 1800 50  0001 C CNN
+	1    5650 1800
+	1    0    0    -1
+$EndComp
 $EndSCHEMATC

Commit message: Changing to AP1509
Parts:
- removed U3: OKI, MRDT_Devices:OKI_Horizontal, symbol MRDT_Devices:OKI
- added D1: D_Schottky, Diode_SMD:D_0603_1608Metric_Pad1.05x0.95mm_HandSolder, symbol Device:D_Schottky
- added D3, D4, D5: LED, LED_SMD:LED_0603_1608Metric_Pad1.05x0.95mm_HandSolder, symbol Device:LED
- added L1: 47uH, Inductor_SMD:L_0603_1608Metric_Pad1.05x0.95mm_HandSolder, symbol pspice:INDUCTOR
- added R2, R3, R4: 500, LED_SMD:LED_0603_1608Metric_Pad1.05x0.95mm_HandSolder, symbol Device:R_Small
- D2: renamed from D?; footprint (none) -> LED_SMD:LED_0603_1608Metric_Pad1.05x0.95mm_HandSolder
- R1: renamed from R?; value 100 -> 500; footprint (none) -> LED_SMD:LED_0603_1608Metric_Pad1.05x0.95mm_HandSolder
- U3: renamed from U?; footprint (none) -> Package_SO:SOIC-8_3.9x4.9mm_P1.27mm
Connections:
- net labels added: +3.3V, Green, Yellow
- net labels removed: +5V
- wire segments 78 -> 112
Other:
- note added: "LED Indicators"

Commit message: Updated to using buttons/switch
Parts:
- added SW1, SW2, SW3, SW4, SW5, SW6: SW_Push, Button_Switch_SMD:SW_SPST_TL3305A, symbol Switch:SW_Push
- added SW7: SW_SPDT, Button_Switch_THT:SW_CuK_OS102011MA1QN1_SPDT_Angled, symbol Switch:SW_SPDT
Connections:
- net labels added: DIRECTION_SW, M1_SW, M2_SW, M3_SW, M4_SW, M5_SW, M6_SW
- wire segments 112 -> 133
Other:
- note added: "Interface"
Changed lines of the file:
@@
 Wire Notes Line
 	2650 3050 11000 3050
+Text Notes 9650 3350 0    98   ~ 20
+Interface
+$Comp
+L Switch:SW_Push SW1
+U 1 1 5C075679
+P 10000 3750
+F 0 "SW1" H 10000 4035 50  0000 C CNN
+F 1 "SW_Push" H 10000 3944 50  0000 C CNN
+F 2 "Button_Switch_SMD:SW_SPST_TL3305A" H 10000 3950 50  0001 C CNN
+F 3 "" H 10000 3950 50  0001 C CNN
+	1    10000 3750
+	1    0    0    -1
+$EndComp
+$Comp
+L power:+3.3V #PWR0110
+U 1 1 5C0791B0
+P 9500 3750
+F 0 "#PWR0110" H 9500 3600 50  0001 C CNN
+F 1 "+3.3V" H 9515 3923 50  0000 C CNN
+F 2 "" H 9500 3750 50  0001 C CNN
+F 3 "" H 9500 3750 50  0001 C CNN
+	1    9500 3750
+	1    0    0    -1
+$EndComp
+Text GLabel 10400 3750 2    50   Output ~ 0
+M1_SW
+Wire Wire Line
+	10200 3750 10400 3750
+Wire Wire Line
+	9800 3750 9500 3750
+$Comp
+L Switch:SW_Push SW2
+U 1 1 5C08079D
+P 10000 4150
+F 0 "SW2" H 10000 4435 50  0000 C CNN
+F 1 "SW_Push" H 10000 4344 50  0000 C CNN
+F 2 "Button_Switch_SMD:SW_SPST_TL3305A" H 10000 4350 50  0001 C CNN
+F 3 "" H 10000 4350 50  0001 C CNN
+	1    10000 4150
+	1    0    0    -1
+$EndComp
+$Comp
+L power:+3.3V #PWR0111
+U 1 1 5C0807A3
+P 9500 4150
+F 0 "#PWR0111" H 9500 4000 50  0001 C CNN
+F 1 "+3.3V" H 9515 4323 50  0000 C CNN
+F 2 "" H 9500 4150 50  0001 C CNN
+F 3 "" H 9500 4150 50  0001 C CNN
+	1    9500 4150
+	1    0    0    -1
+$EndComp
+Text GLabel 10400 4150 2    50   Output ~ 0
+M2_SW
+Wire Wire Line
+	10200 4150 10400 4150
+Wire Wire Line
+	9800 4150 9500 4150
+$Comp
+L Switch:SW_Push SW3
+U 1 1 5C084527
+P 10000 4550
+F 0 "SW3" H 10000 4835 50  0000 C CNN
+F 1 "SW_Push" H 10000 4744 50  0000 C CNN
+F 2 "Button_Switch_SMD:SW_SPST_TL3305A" H 10000 4750 50  0001 C CNN
+F 3 "" H 10000 4750 50  0001 C CNN
+	1    10000 4550
+	1    0    0    -1
+$EndComp
+$Comp
+L power:+3.3V #PWR0112
+U 1 1 5C08452D
+P 9500 4550
+F 0 "#PWR0112" H 9500 4400 50  0001 C CNN
+F 1 "+3.3V" H 9515 4723 50  0000 C CNN
+F 2 "" H 9500 4550 50  0001 C CNN
+F 3 "" H 9500 4550 50  0001 C CNN
+	1    9500 4550
+	1    0    0    -1
+$EndComp
+Text GLabel 10400 4550 2    50   Output ~ 0
+M3_SW
+Wire Wire Line
+	10200 4550 10400 4550
+Wire Wire Line
+	9800 4550 9500 4550
+$Comp
+L Switch:SW_Push SW4
+U 1 1 5C084536
+P 10000 4950
+F 0 "SW4" H 10000 5235 50  0000 C CNN
+F 1 "SW_Push" H 10000 5144 50  0000 C CNN
+F 2 "Button_Switch_SMD:SW_SPST_TL3305A" H 10000 5150 50  0001 C CNN
+F 3 "" H 10000 5150 50  0001 C CNN
+	1    10000 4950
+	1    0    0    -1
+$EndComp
+$Comp
+L power:+3.3V #PWR0113
+U 1 1 5C08453C
+P 9500 4950
+F 0 "#PWR0113" H 9500 4800 50  0001 C CNN
+F 1 "+3.3V" H 9515 5123 50  0000 C CNN
+F 2 "" H 9500 4950 50  0001 C CNN
+F 3 "" H 9500 4950 50  0001 C CNN
+	1    9500 4950
+	1    0    0    -1
+$EndComp
+Text GLabel 10400 4950 2    50   Output ~ 0
+M4_SW
+Wire Wire Line
+	10200 4950 10400 4950
+Wire Wire Line
+	9800 4950 9500 4950
+$Comp
+L Switch:SW_Push SW5
+U 1 1 5C0886D5
+P 10000 5300
+F 0 "SW5" H 10000 5585 50  0000 C CNN
+F 1 "SW_Push" H 10000 5494 50  0000 C CNN
+F 2 "Button_Switch_SMD:SW_SPST_TL3305A" H 10000 5500 50  0001 C CNN
+F 3 "" H 10000 5500 50  0001 C CNN
+	1    10000 5300
+	1    0    0    -1
+$EndComp
+$Comp
+L power:+3.3V #PWR0114
+U 1 1 5C0886DB
+P 9500 5300
+F 0 "#PWR0114" H 9500 5150 50  0001 C CNN
+F 1 "+3.3V" H 9515 5473 50  0000 C CNN
+F 2 "" H 9500 5300 50  0001 C CNN
+F 3 "" H 9500 5300 50  0001 C CNN
+	1    9500 5300
+	1    0    0    -1
+$EndComp
+Text GLabel 10400 5300 2    50   Output ~ 0
+M5_SW
+Wire Wire Line
+	10200 5300 10400 5300
+Wire Wire Line
+	9800 5300 9500 5300
+$Comp
+L Switch:SW_Push SW6
+U 1 1 5C0886E4
+P 10000 5700
+F 0 "SW6" H 10000 5985 50  0000 C CNN
+F 1 "SW_Push" H 10000 5894 50  0000 C CNN
+F 2 "Button_Switch_SMD:SW_SPST_TL3305A" H 10000 5900 50  0001 C CNN
+F 3 "" H 10000 5900 50  0001 C CNN
+	1    10000 5700
+	1    0    0    -1
+$EndComp
+$Comp
+L power:+3.3V #PWR0115
+U 1 1 5C0886EA
+P 9500 5700
+F 0 "#PWR0115" H 9500 5550 50  0001 C CNN
+F 1 "+3.3V" H 9515 5873 50  0000 C CNN
+F 2 "" H 9500 5700 50  0001 C CNN
+F 3 "" H 9500 5700 50  0001 C CNN
+	1    9500 5700
+	1    0    0    -1
+$EndComp
+Text GLabel 10400 5700 2    50   Output ~ 0
+M6_SW
+Wire Wire Line
+	10200 5700 10400 5700
+Wire Wire Line
+	9800 5700 9500 5700
+$Comp
+L Switch:SW_SPDT SW7
+U 1 1 5C09152C
+P 10000 6100
+F 0 "SW7" H 10000 6385 50  0000 C CNN
+F 1 "SW_SPDT" H 10000 6294 50  0000 C CNN
+F 2 "Button_Switch_THT:SW_CuK_OS102011MA1QN1_SPDT_Angled" H 10000 6100 50  0001 C CNN
+F 3 "" H 10000 6100 50  0001 C CNN
+	1    10000 6100
+	1    0    0    -1
+$EndComp
+$Comp
+L power:+3.3V #PWR0116
+U 1 1 5C091779
+P 9500 6100
+F 0 "#PWR0116" H 9500 5950 50  0001 C CNN
+F 1 "+3.3V" H 9515 6273 50  0000 C CNN
+F 2 "" H 9500 6100 50  0001 C CNN
+F 3 "" H 9500 6100 50  0001 C CNN
+	1    9500 6100
+	1    0    0    -1
+$EndComp
+Wire Wire Line
+	9800 6100 9500 6100
+Text GLabel 10400 6000 2    50   Output ~ 0
+DIRECTION_SW
+Wire Wire Line
+	10200 6000 10400 6000
+Text GLabel 6600 4300 0    50   Input ~ 0
+M1_SW
+Text GLabel 6600 4400 0    50   Input ~ 0
+M2_SW
+Text GLabel 6600 4500 0    50   Input ~ 0
+M3_SW
+Text GLabel 6600 4600 0    50   Input ~ 0
+M4_SW
+Text GLabel 6600 4700 0    50   Input ~ 0
+M5_SW
+Text GLabel 6600 4800 0    50   Input ~ 0
+M6_SW
+Text GLabel 6600 4000 0    50   Input ~ 0
+DIRECTION_SW
+Wire Wire Line
+	6850 4000 6600 4000
+Wire Wire Line
+	6600 4300 6850 4300
+Wire Wire Line
+	6850 4400 6600 4400
+Wire Wire Line
+	6600 4500 6850 4500
+Wire Wire Line
+	6850 4600 6600 4600
+Wire Wire Line
+	6600 4700 6850 4700
+Wire Wire Line
+	6850 4800 6600 4800
 $EndSCHEMATC

Commit message: changes to schematic and starting changes to layout
Parts:
- removed C1, C10, C11, C12, C2, C3, C4, C5, C6, C9: .1uF, Capacitor_SMD:C_0603_1608Metric_Pad1.05x0.95mm_HandSolder, symbol Device:C
- added C1, C10, C11, C12, C2, C9: .1uF, symbol Device:C_Small
- added C3, C4, C5, C6: 10uF, symbol Device:C_Small
- added D6, D7, D8, D9: LED, LED_SMD:LED_0603_1608Metric_Pad1.05x0.95mm_HandSolder, symbol Device:LED
- added R5, R6, R7, R8: 500, LED_SMD:LED_0603_1608Metric_Pad1.05x0.95mm_HandSolder, symbol Device:R_Small
Connections:
- net labels added: +5V, Lspeed, Power, Rspeed, Watchdog
- net labels removed: +3.3V, Green, Yellow
- wire segments 133 -> 147
Other:
- note added: "Green"
- note added: "Red"
- note added: "Yellow"
