File: DriveBoard_Hardware/DriveBoard_Hardware.sch (KiCad schematic (older format))
At the start: 45 parts, among them SW1 SW_Push, SW2 SW_Push, SW3 SW_Push, SW4 SW_Push, SW5 SW_Push, SW6 SW_Push, SW7 SW_SPDT, U1 MAX_3232, U2 MAX_3232, U3 AP1059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

Commit message: making changes
Parts:
- removed D1: D_Schottky, Diode_SMD:D_0603_1608Metric_Pad1.05x0.95mm_HandSolder, symbol Device:D_Schottky
- removed L1: 47uH, Inductor_SMD:L_0603_1608Metric_Pad1.05x0.95mm_HandSolder, symbol pspice:INDUCTOR
- removed U3: AP1059, Package_SO:SOIC-8_3.9x4.9mm_P1.27mm, symbol MRDT_ICs:AP1059
- added U3: OKI, MRDT_Devices:OKI_Horizontal, symbol MRDT_Devices:OKI
- C1, C10, C11, C12, C2, C3, C4, C5, C6, C9: footprint (none) -> Capacitor_SMD:C_0603_1608Metric_Pad1.05x0.95mm_HandSolder
Connections:
- wire segments 147 -> 126
Other:
- moved on the sheet: C7, C8, Conn1A, Conn1B
Changed lines of the file:
@@
 L MRDT_Connectors:AndersonPP Conn1
 U 1 1 5BC68926
-P 2800 2700
-F 0 "Conn1" H 3006 2981 60  0000 C CNN
-F 1 "AndersonPP" H 3006 2981 60  0001 C CNN
-F 2 "MRDT_Connectors:Anderson_2_Horisontal_Side_by_Side" H 2650 2150 60  0001 C CNN
-F 3 "" H 2650 2150 60  0001 C CNN
-	1    2800 2700
+P 3150 2200
+F 0 "Conn1" H 3300 2450 60  0000 C CNN
+F 1 "AndersonPP" H 3356 2481 60  0001 C CNN
+F 2 "MRDT_Connectors:Anderson_2_Horisontal_Side_by_Side" H 3000 1650 60  0001 C CNN
+F 3 "" H 3000 1650 60  0001 C CNN
+	1    3150 2200
 	1    0    0    -1
 $EndComp
@@
 L Device:C C7
 U 1 1 5BC69222
-P 3350 1700
-F 0 "C7" H 3150 1750 50  0000 L CNN
-F 1 "10uF" H 3050 1650 50  0000 L CNN
-F 2 "Capacitor_SMD:C_0603_1608Metric_Pad1.05x0.95mm_HandSolder" H 3388 1550 50  0001 C CNN
-F 3 "~" H 3350 1700 50  0001 C CNN
-	1    3350 1700
+P 3850 1950
+F 0 "C7" H 3650 2000 50  0000 L CNN
+F 1 "10uF" H 3550 1900 50  0000 L CNN
+F 2 "Capacitor_SMD:C_0603_1608Metric_Pad1.05x0.95mm_HandSolder" H 3888 1800 50  0001 C CNN
+F 3 "~" H 3850 1950 50  0001 C CNN
+	1    3850 1950
 	1    0    0    -1
 $EndComp
@@
 L Device:C C8
 U 1 1 5BC69286
-P 4750 2450
-F 0 "C8" H 4865 2496 50  0000 L CNN
-F 1 "10uF" H 4865 2405 50  0000 L CNN
-F 2 "Capacitor_SMD:C_0603_1608Metric_Pad1.05x0.95mm_HandSolder" H 4788 2300 50  0001 C CNN
-F 3 "~" H 4750 2450 50  0001 C CNN
-	1    4750 2450
+P 5100 1950
+F 0 "C8" H 5215 1996 50  0000 L CNN
+F 1 "10uF" H 5215 1905 50  0000 L CNN
+F 2 "Capacitor_SMD:C_0603_1608Metric_Pad1.05x0.95mm_HandSolder" H 5138 1800 50  0001 C CNN
+F 3 "~" H 5100 1950 50  0001 C CNN
+	1    5100 1950
 	1    0    0    -1
 $EndComp
@@
 L power:GND #PWR06
 U 1 1 5BC693BC
-P 5100 2600
-F 0 "#PWR06" H 5100 2350 50  0001 C CNN
-F 1 "GND" H 5105 2427 50  0000 C CNN
-F 2 "" H 5100 2600 50  0001 C CNN
-F 3 "" H 5100 2600 50  0001 C CNN
-	1    5100 2600
-	1    0    0    -1
-$EndComp
-Wire Wire Line
-	4750 2600 5100 2600
+P 5450 2100
+F 0 "#PWR06" H 5450 1850 50  0001 C CNN
+F 1 "GND" H 5455 1927 50  0000 C CNN
+F 2 "" H 5450 2100 50  0001 C CNN
+F 3 "" H 5450 2100 50  0001 C CNN
+	1    5450 2100
+	1    0    0    -1
+$EndComp
+Wire Wire Line
+	5100 2100 5450 2100
 $Comp
 L MRDT_ICs:MAX_3232 U1
@@
 Serial 6
 $Comp
-L MRDT_ICs:AP1059 U3
-U 1 1 5BE8A9F0
-P 3900 1900
-F 0 "U3" H 4125 2497 60  0000 C CNN
-F 1 "AP1059" H 4125 2391 60  0000 C CNN
-F 2 "Package_SO:SOIC-8_3.9x4.9mm_P1.27mm" H 3650 1800 60  0001 C CNN
-F 3 "" H 3650 1800 60  0001 C CNN
-	1    3900 1900
-	1    0    0    -1
-$EndComp
-$Comp
 L Device:LED D2
 U 1 1 5BE8AD8F
@@
 	-1   0    0    1
 $EndComp
-$Comp
-L Device:D_Schottky D1
-U 1 1 5C00F090
-P 3600 2400
-F 0 "D1" V 3554 2479 50  0000 L CNN
-F 1 "D_Schottky" V 3645 2479 50  0000 L CNN
-F 2 "Diode_SMD:D_0603_1608Metric_Pad1.05x0.95mm_HandSolder" H 3600 2400 50  0001 C CNN
-F 3 "~" H 3600 2400 50  0001 C CNN
-	1    3600 2400
-	0    1    1    0
-$EndComp
-Wire Wire Line
-	3700 1550 3350 1550
-Wire Wire Line
-	3700 1850 3350 1850
-Wire Wire Line
-	4750 2600 4600 2600
-Wire Wire Line
-	3350 2600 3350 1850
-Connection ~ 4750 2600
-Connection ~ 3350 1850
-Wire Wire Line
-	3200 2600 3350 2600
-Connection ~ 3350 2600
-$Comp
-L pspice:INDUCTOR L1
-U 1 1 5C041C84
-P 4100 2150
-F 0 "L1" H 4100 2000 50  0000 C CNN
-F 1 "47uH" H 4100 2100 50  0000 C CNN
-F 2 "Inductor_SMD:L_0603_1608Metric_Pad1.05x0.95mm_HandSolder" H 4100 2150 50  0001 C CNN
-F 3 "" H 4100 2150 50  0001 C CNN
-	1    4100 2150
-	1    0    0    -1
-$EndComp
-Wire Wire Line
-	3700 1650 3600 1650
-Wire Wire Line
-	3600 1650 3600 2150
-Wire Wire Line
-	3600 2150 3850 2150
-Wire Wire Line
-	3600 2250 3600 2150
-Connection ~ 3600 2150
-Wire Wire Line
-	3600 2550 3600 2600
-Connection ~ 3600 2600
-Wire Wire Line
-	3600 2600 3350 2600
-Wire Wire Line
-	4350 2150 4750 2150
-Wire Wire Line
-	4750 2150 4750 2300
-Connection ~ 4750 2150
-Wire Wire Line
-	4550 1850 4600 1850
-Wire Wire Line
-	4600 1850 4600 2600
-Connection ~ 4600 2600
-Wire Wire Line
-	4600 2600 3600 2600
-Wire Wire Line
-	4550 1750 4600 1750
-Wire Wire Line
-	4600 1750 4600 1850
-Connection ~ 4600 1850
-Wire Wire Line
-	4550 1650 4600 1650
-Wire Wire Line
-	4600 1650 4600 1750
-Connection ~ 4600 1750
-Wire Wire Line
-	4550 1550 4600 1550
-Wire Wire Line
-	4600 1550 4600 1650
-Connection ~ 4600 1650
-Wire Wire Line
-	4750 2150 4750 1950
-Wire Wire Line
-	4750 1950 3650 1950
-Wire Wire Line
-	3650 1950 3650 1750
-Wire Wire Line
-	3650 1750 3700 1750
-Text Label 3350 1550 0    50   ~ 0
+Connection ~ 5100 2100
+Text Label 3600 1800 0    50   ~ 0
 +12V
 $Comp
@@
 Wire Wire Line
 	9700 1950 9700 2050
-Wire Wire Line
-	4750 2150 5650 2150
 $Comp
 L Device:R_Small R3
@@
 L power:+5V #PWR0101
 U 1 1 5C147F3B
-P 5650 2150
-F 0 "#PWR0101" H 5650 2000 50  0001 C CNN
-F 1 "+5V" H 5665 2323 50  0000 C CNN
-F 2 "" H 5650 2150 50  0001 C CNN
-F 3 "" H 5650 2150 50  0001 C CNN
-	1    5650 2150
+P 5450 1800
+F 0 "#PWR0101" H 5450 1650 50  0001 C CNN
+F 1 "+5V" H 5465 1973 50  0000 C CNN
+F 2 "" H 5450 1800 50  0001 C CNN
+F 3 "" H 5450 1800 50  0001 C CNN
+	1    5450 1800
 	1    0    0    -1
 $EndComp
@@
 L MRDT_Connectors:AndersonPP Conn1
 U 2 1 5BC68A39
-P 2800 1650
-F 0 "Conn1" H 3006 1931 60  0000 C CNN
-F 1 "AndersonPP" H 3006 1931 60  0001 C CNN
-F 2 "MRDT_Connectors:Anderson_2_Horisontal_Side_by_Side" H 2650 1100 60  0001 C CNN
-F 3 "" H 2650 1100 60  0001 C CNN
-	2    2800 1650
-	1    0    0    -1
-$EndComp
-Wire Wire Line
-	3350 1550 3200 1550
-Connection ~ 3350 1550
+P 3150 1900
+F 0 "Conn1" H 3300 2150 60  0000 C CNN
+F 1 "AndersonPP" H 3356 2181 60  0001 C CNN
+F 2 "MRDT_Connectors:Anderson_2_Horisontal_Side_by_Side" H 3000 1350 60  0001 C CNN
+F 3 "" H 3000 1350 60  0001 C CNN
+	2    3150 1900
+	1    0    0    -1
+$EndComp
 $Comp
 L Device:C_Small C9
@@
 F 0 "C9" H 5058 3754 50  0000 R CNN
 F 1 ".1uF" H 5058 3845 50  0000 R CNN
-F 2 "" H 5150 3800 50  0001 C CNN
+F 2 "Capacitor_SMD:C_0603_1608Metric_Pad1.05x0.95mm_HandSolder" H 5150 3800 50  0001 C CNN
 F 3 "~" H 5150 3800 50  0001 C CNN
 	1    5150 3800
@@
 F 0 "C10" H 5058 4054 50  0000 R CNN
 F 1 ".1uF" H 5058 4145 50  0000 R CNN
-F 2 "" H 5150 4100 50  0001 C CNN
+F 2 "Capacitor_SMD:C_0603_1608Metric_Pad1.05x0.95mm_HandSolder" H 5150 4100 50  0001 C CNN
 F 3 "~" H 5150 4100 50  0001 C CNN
 	1    5150 4100
@@
 F 0 "C1" H 3308 3754 50  0000 R CNN
 F 1 ".1uF" H 3308 3845 50  0000 R CNN
-F 2 "" H 3400 3800 50  0001 C CNN
+F 2 "Capacitor_SMD:C_0603_1608Metric_Pad1.05x0.95mm_HandSolder" H 3400 3800 50  0001 C CNN
 F 3 "~" H 3400 3800 50  0001 C CNN
 	1    3400 3800
@@
 F 0 "C2" H 3308 5254 50  0000 R CNN
 F 1 ".1uF" H 3308 5345 50  0000 R CNN
-F 2 "" H 3400 5300 50  0001 C CNN
+F 2 "Capacitor_SMD:C_0603_1608Metric_Pad1.05x0.95mm_HandSolder" H 3400 5300 50  0001 C CNN
 F 3 "~" H 3400 5300 50  0001 C CNN
 	1    3400 5300
@@
 F 0 "C3" V 3550 4200 50  0000 C CNN
 F 1 "10uF" V 3550 3950 50  0000 C CNN
-F 2 "" H 3500 4100 50  0001 C CNN
+F 2 "Capacitor_SMD:C_0603_1608Metric_Pad1.05x0.95mm_HandSolder" H 3500 4100 50  0001 C CNN
 F 3 "~" H 3500 4100 50  0001 C CNN
 	1    3500 4100
@@
 F 0 "C4" V 3450 4300 50  0000 C CNN
 F 1 "10uF" V 3450 4050 50  0000 C CNN
-F 2 "" H 3500 4200 50  0001 C CNN
+F 2 "Capacitor_SMD:C_0603_1608Metric_Pad1.05x0.95mm_HandSolder" H 3500 4200 50  0001 C CNN
 F 3 "~" H 3500 4200 50  0001 C CNN
 	1    3500 4200
@@
 F 0 "C11" H 5058 5254 50  0000 R CNN
 F 1 ".1uF" H 5058 5345 50  0000 R CNN
-F 2 "" H 5150 5300 50  0001 C CNN
+F 2 "Capacitor_SMD:C_0603_1608Metric_Pad1.05x0.95mm_HandSolder" H 5150 5300 50  0001 C CNN
 F 3 "~" H 5150 5300 50  0001 C CNN
 	1    5150 5300
@@
 F 0 "C12" H 5058 5554 50  0000 R CNN
 F 1 ".1uF" H 5058 5645 50  0000 R CNN
-F 2 "" H 5150 5600 50  0001 C CNN
+F 2 "Capacitor_SMD:C_0603_1608Metric_Pad1.05x0.95mm_HandSolder" H 5150 5600 50  0001 C CNN
 F 3 "~" H 5150 5600 50  0001 C CNN
 	1    5150 5600
@@
 F 0 "C6" V 3450 5800 50  0000 C CNN
 F 1 "10uF" V 3450 5550 50  0000 C CNN
-F 2 "" H 3500 5700 50  0001 C CNN
+F 2 "Capacitor_SMD:C_0603_1608Metric_Pad1.05x0.95mm_HandSolder" H 3500 5700 50  0001 C CNN
 F 3 "~" H 3500 5700 50  0001 C CNN
 	1    3500 5700
@@
 F 0 "C5" V 3550 5700 50  0000 C CNN
 F 1 "10uF" V 3550 5450 50  0000 C CNN
-F 2 "" H 3500 5600 50  0001 C CNN
+F 2 "Capacitor_SMD:C_0603_1608Metric_Pad1.05x0.95mm_HandSolder" H 3500 5600 50  0001 C CNN
 F 3 "~" H 3500 5600 50  0001 C CNN
 	1    3500 5600
@@
 Wire Wire Line
 	7900 3900 7750 3900
+Wire Wire Line
+	3550 2100 3850 2100
+$Comp
+L MRDT_Devices:OKI U3
+U 1 1 5C167EEB
+P 4150 1900
+F 0 "U3" H 4200 1850 60  0001 C CNN
+F 1 "OKI" H 4350 2181 60  0000 C CNN
+F 2 "MRDT_Devices:OKI_Horizontal" H 3950 1800 60  0001 C CNN
+F 3 "" H 3950 1800 60  0001 C CNN
+	1    4150 1900
+	1    0    0    -1
+$EndComp
+Connection ~ 4350 2100
+Wire Wire Line
+	4350 2100 5100 2100
+Wire Wire Line
+	4750 1800 5100 1800
+Connection ~ 3850 2100
+Wire Wire Line
+	3850 2100 4350 2100
+Wire Wire Line
+	3950 1800 3850 1800
+Wire Wire Line
+	3550 1800 3850 1800
+Connection ~ 3850 1800
+Wire Wire Line
+	5100 1800 5450 1800
+Connection ~ 5100 1800
 $EndSCHEMATC

Commit message: finishing changes
Parts:
- removed D9: LED, LED_SMD:LED_0603_1608Metric_Pad1.05x0.95mm_HandSolder, symbol Device:LED
- removed R8: 500, LED_SMD:LED_0603_1608Metric_Pad1.05x0.95mm_HandSolder, symbol Device:R_Small
Connections:
- net labels removed: Power
- wire segments 126 -> 122
Other:
- moved on the sheet: D6, D7, D8, R5, R6, R7
Changed lines of the file:
@@
 Wire Wire Line
 	10550 2050 10550 1950
-Text Notes 8800 800  0    98   ~ 20
+Text Notes 8850 750  0    98   ~ 20
 LED Indicators
 Wire Notes Line
@@
 Text Notes 9150 2350 0    50   ~ 0
 Green
-Text GLabel 7900 4100 2    50   Output ~ 0
-Power
 Wire Wire Line
 	7750 4000 8400 4000
-Wire Wire Line
-	7900 4100 7750 4100
 Wire Wire Line
 	7900 4500 7750 4500
@@
 	7800 3050 7800 550
 $Comp
-L Device:R_Small R8
-U 1 1 5C22B85D
+L Device:R_Small R7
+U 1 1 5C2312DF
 P 8900 1450
-F 0 "R8" V 9000 1400 50  0000 L CNN
+F 0 "R7" V 9000 1400 50  0000 L CNN
 F 1 "500" V 8800 1400 50  0000 L CNN
 F 2 "LED_SMD:LED_0603_1608Metric_Pad1.05x0.95mm_HandSolder" H 8900 1450 50  0001 C CNN
@@
 $EndComp
 $Comp
-L Device:LED D9
-U 1 1 5C22B863
+L Device:LED D8
+U 1 1 5C2312E5
 P 8900 1800
-F 0 "D9" H 8950 1900 50  0000 R CNN
+F 0 "D8" H 8950 1900 50  0000 R CNN
 F 1 "LED" H 8950 1700 50  0000 R CNN
 F 2 "LED_SMD:LED_0603_1608Metric_Pad1.05x0.95mm_HandSolder" H 8900 1800 50  0001 C CNN
@@
 $EndComp
 $Comp
-L power:GND #PWR0117
-U 1 1 5C22B869
+L power:GND #PWR0118
+U 1 1 5C2312EB
 P 8900 2050
-F 0 "#PWR0117" H 8900 1800 50  0001 C CNN
+F 0 "#PWR0118" H 8900 1800 50  0001 C CNN
 F 1 "GND" H 8905 1877 50  0000 C CNN
 F 2 "" H 8900 2050 50  0001 C CNN
@@
 	8900 2050 8900 1950
 $Comp
-L Device:R_Small R7
-U 1 1 5C2312DF
+L Device:R_Small R6
+U 1 1 5C2428F7
 P 8600 1450
-F 0 "R7" V 8700 1400 50  0000 L CNN
+F 0 "R6" V 8700 1400 50  0000 L CNN
 F 1 "500" V 8500 1400 50  0000 L CNN
 F 2 "LED_SMD:LED_0603_1608Metric_Pad1.05x0.95mm_HandSolder" H 8600 1450 50  0001 C CNN
@@
 $EndComp
 $Comp
-L Device:LED D8
-U 1 1 5C2312E5
+L Device:LED D7
+U 1 1 5C2428FD
 P 8600 1800
-F 0 "D8" H 8650 1900 50  0000 R CNN
+F 0 "D7" H 8650 1900 50  0000 R CNN
 F 1 "LED" H 8650 1700 50  0000 R CNN
 F 2 "LED_SMD:LED_0603_1608Metric_Pad1.05x0.95mm_HandSolder" H 8600 1800 50  0001 C CNN
@@
 $EndComp
 $Comp
-L power:GND #PWR0118
-U 1 1 5C2312EB
+L power:GND #PWR0119
+U 1 1 5C242903
 P 8600 2050
-F 0 "#PWR0118" H 8600 1800 50  0001 C CNN
+F 0 "#PWR0119" H 8600 1800 50  0001 C CNN
 F 1 "GND" H 8605 1877 50  0000 C CNN
 F 2 "" H 8600 2050 50  0001 C CNN
@@
 	8600 2050 8600 1950
 $Comp
-L Device:R_Small R6
-U 1 1 5C2428F7
+L Device:R_Small R5
+U 1 1 5C24290E
 P 8300 1450
-F 0 "R6" V 8400 1400 50  0000 L CNN
+F 0 "R5" V 8400 1400 50  0000 L CNN
 F 1 "500" V 8200 1400 50  0000 L CNN
 F 2 "LED_SMD:LED_0603_1608Metric_Pad1.05x0.95mm_HandSolder" H 8300 1450 50  0001 C CNN
@@
 $EndComp
 $Comp
-L Device:LED D7
-U 1 1 5C2428FD
+L Device:LED D6
+U 1 1 5C242914
 P 8300 1800
-F 0 "D7" H 8350 1900 50  0000 R CNN
+F 0 "D6" H 8350 1900 50  0000 R CNN
 F 1 "LED" H 8350 1700 50  0000 R CNN
 F 2 "LED_SMD:LED_0603_1608Metric_Pad1.05x0.95mm_HandSolder" H 8300 1800 50  0001 C CNN
@@
 $EndComp
 $Comp
-L power:GND #PWR0119
-U 1 1 5C242903
+L power:GND #PWR0120
+U 1 1 5C24291A
 P 8300 2050
-F 0 "#PWR0119" H 8300 1800 50  0001 C CNN
+F 0 "#PWR0120" H 8300 1800 50  0001 C CNN
 F 1 "GND" H 8305 1877 50  0000 C CNN
 F 2 "" H 8300 2050 50  0001 C CNN
@@
 Wire Wire Line
 	8300 2050 8300 1950
-$Comp
-L Device:R_Small R5
-U 1 1 5C24290E
-P 8000 1450
-F 0 "R5" V 8100 1400 50  0000 L CNN
-F 1 "500" V 7900 1400 50  0000 L CNN
-F 2 "LED_SMD:LED_0603_1608Metric_Pad1.05x0.95mm_HandSolder" H 8000 1450 50  0001 C CNN
-F 3 "~" H 8000 1450 50  0001 C CNN
-	1    8000 1450
-	-1   0    0    1
-$EndComp
-$Comp
-L Device:LED D6
-U 1 1 5C242914
-P 8000 1800
-F 0 "D6" H 8050 1900 50  0000 R CNN
-F 1 "LED" H 8050 1700 50  0000 R CNN
-F 2 "LED_SMD:LED_0603_1608Metric_Pad1.05x0.95mm_HandSolder" H 8000 1800 50  0001 C CNN
-F 3 "~" H 8000 1800 50  0001 C CNN
-	1    8000 1800
-	0    -1   -1   0
-$EndComp
-$Comp
-L power:GND #PWR0120
-U 1 1 5C24291A
-P 8000 2050
-F 0 "#PWR0120" H 8000 1800 50  0001 C CNN
-F 1 "GND" H 8005 1877 50  0000 C CNN
-F 2 "" H 8000 2050 50  0001 C CNN
-F 3 "" H 8000 2050 50  0001 C CNN
-	1    8000 2050
-	1    0    0    -1
-$EndComp
-Wire Wire Line
-	8000 1550 8000 1650
-Wire Wire Line
-	8000 2050 8000 1950
-Text Notes 8800 2350 0    50   ~ 0
-Green
-Text Notes 8550 2350 0    50   ~ 0
+Text Notes 8850 2350 0    50   ~ 0
 Red
+Text Notes 8500 2350 0    50   ~ 0
+Yellow
 Text Notes 8200 2350 0    50   ~ 0
 Yellow
-Text Notes 7900 2350 0    50   ~ 0
-Yellow
-Text GLabel 8000 1150 1    50   Input ~ 0
+Text GLabel 8300 1150 1    50   Input ~ 0
 Lspeed
-Text GLabel 8300 1150 1    50   Input ~ 0
+Text GLabel 8600 1150 1    50   Input ~ 0
 Rspeed
 Wire Wire Line
+	8600 1150 8600 1350
+Wire Wire Line
 	8300 1150 8300 1350
-Wire Wire Line
-	8000 1150 8000 1350
-Text GLabel 8900 1150 1    50   Input ~ 0
-Power
-Wire Wire Line
-	8900 1150 8900 1350
-Text GLabel 8600 1200 1    50   Input ~ 0
+Text GLabel 8900 1200 1    50   Input ~ 0
 Watchdog
 Wire Wire Line
-	8600 1200 8600 1350
+	8900 1200 8900 1350
 Wire Wire Line
 	7750 4200 7900 4200

Commit message: updating changes (Rev1 Review)
Parts:
- added R10, R11, R12, R13, R14, R8, R9: 10K, Resistor_SMD:R_0603_1608Metric_Pad1.05x0.95mm_HandSolder, symbol Device:R
Connections:
- wire segments 122 -> 149
Changed lines of the file:
@@
 M1_SW
 Wire Wire Line
-	10200 3750 10400 3750
+	10200 3750 10300 3750
 Wire Wire Line
 	9800 3750 9500 3750
@@
 M2_SW
 Wire Wire Line
-	10200 4150 10400 4150
+	10200 4150 10300 4150
 Wire Wire Line
 	9800 4150 9500 4150
@@
 M3_SW
 Wire Wire Line
-	10200 4550 10400 4550
+	10200 4550 10300 4550
 Wire Wire Line
 	9800 4550 9500 4550
@@
 M4_SW
 Wire Wire Line
-	10200 4950 10400 4950
+	10200 4950 10300 4950
 Wire Wire Line
 	9800 4950 9500 4950
@@
 M5_SW
 Wire Wire Line
-	10200 5300 10400 5300
+	10200 5300 10300 5300
 Wire Wire Line
 	9800 5300 9500 5300
@@
 M6_SW
 Wire Wire Line
-	10200 5700 10400 5700
+	10200 5700 10300 5700
 Wire Wire Line
 	9800 5700 9500 5700
@@
 DIRECTION_SW
 Wire Wire Line
-	10200 6000 10400 6000
+	10200 6000 10300 6000
 Text GLabel 7900 4500 2    50   Input ~ 0
 M1_SW
@@
 	5100 1800 5450 1800
 Connection ~ 5100 1800
+$Comp
+L Device:R R8
+U 1 1 5C174B63
+P 10450 3950
+F 0 "R8" V 10450 3950 50  0000 C CNN
+F 1 "10K" V 10350 3950 50  0000 C CNN
+F 2 "Resistor_SMD:R_0603_1608Metric_Pad1.05x0.95mm_HandSolder" V 10380 3950 50  0001 C CNN
+F 3 "~" H 10450 3950 50  0001 C CNN
+	1    10450 3950
+	0    1    1    0
+$EndComp
+$Comp
+L power:GND #PWR0117
+U 1 1 5C179CAE
+P 10800 3950
+F 0 "#PWR0117" H 10800 3700 50  0001 C CNN
+F 1 "GND" H 10805 3777 50  0000 C CNN
+F 2 "" H 10800 3950 50  0001 C CNN
+F 3 "" H 10800 3950 50  0001 C CNN
+	1    10800 3950
+	1    0    0    -1
+$EndComp
+Wire Wire Line
+	10800 3950 10600 3950
+Wire Wire Line
+	10300 3950 10300 3750
+Connection ~ 10300 3750
+Wire Wire Line
+	10300 3750 10400 3750
+$Comp
+L Device:R R9
+U 1 1 5C188834
+P 10500 4350
+F 0 "R9" V 10500 4350 50  0000 C CNN
+F 1 "10K" V 10400 4350 50  0000 C CNN
+F 2 "Resistor_SMD:R_0603_1608Metric_Pad1.05x0.95mm_HandSolder" V 10430 4350 50  0001 C CNN
+F 3 "~" H 10500 4350 50  0001 C CNN
+	1    10500 4350
+	0    1    1    0
+$EndComp
+$Comp
+L power:GND #PWR0121
+U 1 1 5C18883A
+P 10850 4350
+F 0 "#PWR0121" H 10850 4100 50  0001 C CNN
+F 1 "GND" H 10855 4177 50  0000 C CNN
+F 2 "" H 10850 4350 50  0001 C CNN
+F 3 "" H 10850 4350 50  0001 C CNN
+	1    10850 4350
+	1    0    0    -1
+$EndComp
+Wire Wire Line
+	10850 4350 10650 4350
+$Comp
+L Device:R R10
+U 1 1 5C18D796
+P 10500 4750
+F 0 "R10" V 10500 4750 50  0000 C CNN
+F 1 "10K" V 10400 4750 50  0000 C CNN
+F 2 "Resistor_SMD:R_0603_1608Metric_Pad1.05x0.95mm_HandSolder" V 10430 4750 50  0001 C CNN
+F 3 "~" H 10500 4750 50  0001 C CNN
+	1    10500 4750
+	0    1    1    0
+$EndComp
+$Comp
+L power:GND #PWR0122
+U 1 1 5C18D79C
+P 10850 4750
+F 0 "#PWR0122" H 10850 4500 50  0001 C CNN
+F 1 "GND" H 10855 4577 50  0000 C CNN
+F 2 "" H 10850 4750 50  0001 C CNN
+F 3 "" H 10850 4750 50  0001 C CNN
+	1    10850 4750
+	1    0    0    -1
+$EndComp
+Wire Wire Line
+	10850 4750 10650 4750
+$Comp
+L Device:R R11
+U 1 1 5C192938
+P 10500 5150
+F 0 "R11" V 10500 5150 50  0000 C CNN
+F 1 "10K" V 10400 5150 50  0000 C CNN
+F 2 "Resistor_SMD:R_0603_1608Metric_Pad1.05x0.95mm_HandSolder" V 10430 5150 50  0001 C CNN
+F 3 "~" H 10500 5150 50  0001 C CNN
+	1    10500 5150
+	0    1    1    0
+$EndComp
+$Comp
+L power:GND #PWR0123
+U 1 1 5C19293E
+P 10850 5150
+F 0 "#PWR0123" H 10850 4900 50  0001 C CNN
+F 1 "GND" H 10855 4977 50  0000 C CNN
+F 2 "" H 10850 5150 50  0001 C CNN
+F 3 "" H 10850 5150 50  0001 C CNN
+	1    10850 5150
+	1    0    0    -1
+$EndComp
+Wire Wire Line
+	10850 5150 10650 5150
+$Comp
+L Device:R R12
+U 1 1 5C19CEBD
+P 10500 5550
+F 0 "R12" V 10500 5550 50  0000 C CNN
+F 1 "10K" V 10400 5550 50  0000 C CNN
+F 2 "Resistor_SMD:R_0603_1608Metric_Pad1.05x0.95mm_HandSolder" V 10430 5550 50  0001 C CNN
+F 3 "~" H 10500 5550 50  0001 C CNN
+	1    10500 5550
+	0    1    1    0
+$EndComp
+$Comp
+L power:GND #PWR0124
+U 1 1 5C19CEC3
+P 10850 5550
+F 0 "#PWR0124" H 10850 5300 50  0001 C CNN
+F 1 "GND" H 10855 5377 50  0000 C CNN
+F 2 "" H 10850 5550 50  0001 C CNN
+F 3 "" H 10850 5550 50  0001 C CNN
+	1    10850 5550
+	1    0    0    -1
+$EndComp
+Wire Wire Line
+	10850 5550 10650 5550
+$Comp
+L Device:R R13
+U 1 1 5C1A2293
+P 10750 5900
+F 0 "R13" V 10750 5900 50  0000 C CNN
+F 1 "10K" V 10650 5900 50  0000 C CNN
+F 2 "Resistor_SMD:R_0603_1608Metric_Pad1.05x0.95mm_HandSolder" V 10680 5900 50  0001 C CNN
+F 3 "~" H 10750 5900 50  0001 C CNN
+	1    10750 5900
+	0    1    1    0
+$EndComp
+$Comp
+L power:GND #PWR0125
+U 1 1 5C1A2299
+P 11100 5900
+F 0 "#PWR0125" H 11100 5650 50  0001 C CNN
+F 1 "GND" H 11105 5727 50  0000 C CNN
+F 2 "" H 11100 5900 50  0001 C CNN
+F 3 "" H 11100 5900 50  0001 C CNN
+	1    11100 5900
+	1    0    0    -1
+$EndComp
+Wire Wire Line
+	11100 5900 10900 5900
+Wire Wire Line
+	10600 5900 10300 5900
+Wire Wire Line
+	10300 5900 10300 5700
+Connection ~ 10300 5700
+Wire Wire Line
+	10300 5700 10400 5700
+Wire Wire Line
+	10350 5550 10300 5550
+Wire Wire Line
+	10300 5550 10300 5300
+Connection ~ 10300 5300
+Wire Wire Line
+	10300 5300 10400 5300
+$Comp
+L Device:R R14
+U 1 1 5C1B23AC
+P 10750 6200
+F 0 "R14" V 10750 6200 50  0000 C CNN
+F 1 "10K" V 10650 6200 50  0000 C CNN
+F 2 "Resistor_SMD:R_0603_1608Metric_Pad1.05x0.95mm_HandSolder" V 10680 6200 50  0001 C CNN
+F 3 "~" H 10750 6200 50  0001 C CNN
+	1    10750 6200
+	0    1    1    0
+$EndComp
+$Comp
+L power:GND #PWR0126
+U 1 1 5C1B23B2
+P 11100 6200
+F 0 "#PWR0126" H 11100 5950 50  0001 C CNN
+F 1 "GND" H 11105 6027 50  0000 C CNN
+F 2 "" H 11100 6200 50  0001 C CNN
+F 3 "" H 11100 6200 50  0001 C CNN
+	1    11100 6200
+	1    0    0    -1
+$EndComp
+Wire Wire Line
+	11100 6200 10900 6200
+Wire Wire Line
+	10600 6200 10300 6200
+Wire Wire Line
+	10300 6200 10300 6000
+Connection ~ 10300 6000
+Wire Wire Line
+	10300 6000 10400 6000
+Wire Wire Line
+	10350 5150 10300 5150
+Wire Wire Line
+	10300 5150 10300 4950
+Connection ~ 10300 4950
+Wire Wire Line
+	10300 4950 10400 4950
+Wire Wire Line
+	10350 4750 10300 4750
+Wire Wire Line
+	10300 4750 10300 4550
+Connection ~ 10300 4550
+Wire Wire Line
+	10300 4550 10400 4550
+Wire Wire Line
+	10350 4350 10300 4350
+Wire Wire Line
+	10300 4350 10300 4150
+Connection ~ 10300 4150
+Wire Wire Line
+	10300 4150 10400 4150
 $EndSCHEMATC
