File: DriveBoard_Hardware/DriveBoard_Hardware.sch (KiCad schematic (older format))
At the start: 48 parts, among them SW1 SW_Push, SW2 SW_Push, SW3 SW_Push, SW4 SW_Push, SW5 SW_Push, SW6 SW_Push, SW7 SW_SPDT, U1 MAX_3232, U2 MAX_3232, U3 OKI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

Commit message: updated Rev 2 Libraries
Parts:
- Conn1: footprint MRDT_Connectors:Anderson_2_Horisontal_Side_by_Side -> MRDT_Connectors:Anderson_2_Horizontal_Side_by_Side
- U4: footprint MRDT_Shields:TM4C129E_Launchpad_X7_Bottom_SMD -> MRDT_Shields:TM4C129E_Launchpad_X7_SMD_BOTTOM
Changed lines of the file:
@@
 F 0 "Conn1" H 3300 2450 60  0000 C CNN
 F 1 "AndersonPP" H 3356 2481 60  0001 C CNN
-F 2 "MRDT_Connectors:Anderson_2_Horisontal_Side_by_Side" H 3000 1650 60  0001 C CNN
+F 2 "MRDT_Connectors:Anderson_2_Horizontal_Side_by_Side" H 3000 1650 60  0001 C CNN
 F 3 "" H 3000 1650 60  0001 C CNN
 	1    3150 2200
@@
 F 0 "U4" H 7050 4800 60  0000 L CNN
 F 1 "TM4C129E_Launchpad" H 6850 6500 60  0001 L CNN
-F 2 "MRDT_Shields:TM4C129E_Launchpad_X7_Bottom_SMD" H 7050 4850 60  0001 C CNN
+F 2 "MRDT_Shields:TM4C129E_Launchpad_X7_SMD_BOTTOM" H 7050 4850 60  0001 C CNN
 F 3 "" H 7050 4850 60  0001 C CNN
 	5    7050 4850
@@
 F 0 "U4" H 7650 4800 60  0000 C CNN
 F 1 "TM4C129E_Launchpad" H 7750 6050 60  0000 C CNN
-F 2 "MRDT_Shields:TM4C129E_Launchpad_X7_Bottom_SMD" H 7550 4850 60  0001 C CNN
+F 2 "MRDT_Shields:TM4C129E_Launchpad_X7_SMD_BOTTOM" H 7550 4850 60  0001 C CNN
 F 3 "" H 7550 4850 60  0001 C CNN
 	6    7550 4850
@@
 F 0 "U4" H 7050 6100 60  0000 L CNN
 F 1 "TM4C129E_Launchpad" H 7355 6642 60  0001 L CNN
-F 2 "MRDT_Shields:TM4C129E_Launchpad_X7_Bottom_SMD" H 7050 6150 60  0001 C CNN
+F 2 "MRDT_Shields:TM4C129E_Launchpad_X7_SMD_BOTTOM" H 7050 6150 60  0001 C CNN
 F 3 "" H 7050 6150 60  0001 C CNN
 	7    7050 6150
@@
 F 0 "U4" H 7650 6100 60  0000 C CNN
 F 1 "TM4C129E_Launchpad" H 7750 7350 60  0001 C CNN
-F 2 "MRDT_Shields:TM4C129E_Launchpad_X7_Bottom_SMD" H 7550 6150 60  0001 C CNN
+F 2 "MRDT_Shields:TM4C129E_Launchpad_X7_SMD_BOTTOM" H 7550 6150 60  0001 C CNN
 F 3 "" H 7550 6150 60  0001 C CNN
 	8    7550 6150
@@
 F 0 "Conn1" H 3300 2150 60  0000 C CNN
 F 1 "AndersonPP" H 3356 2181 60  0001 C CNN
-F 2 "MRDT_Connectors:Anderson_2_Horisontal_Side_by_Side" H 3000 1350 60  0001 C CNN
+F 2 "MRDT_Connectors:Anderson_2_Horizontal_Side_by_Side" H 3000 1350 60  0001 C CNN
 F 3 "" H 3000 1350 60  0001 C CNN
 	2    3150 1900

Commit message: Created rev 2
Parts:
- removed C10, C11, C12, C9: .1uF, Capacitor_SMD:C_0603_1608Metric_Pad1.05x0.95mm_HandSolder, symbol Device:C_Small
- removed C4, C5, C6: 10uF, Capacitor_SMD:C_0603_1608Metric_Pad1.05x0.95mm_HandSolder, symbol Device:C_Small
- removed U1, U2: MAX_3232, Package_SO:SOIC-16_3.9x9.9mm_P1.27mm, symbol MRDT_ICs:MAX_3232
- added Conn5, Conn6, Conn7: Molex_SL_03, MRDT_Connectors:MOLEX_SL_03_Horizontal, symbol MRDT_Connectors:Molex_SL_03
- added D1, D10, D11, D12, D13, D14, D15, D16, D17, D9: LED, LED_SMD:LED_0603_1608Metric_Pad1.05x0.95mm_HandSolder, symbol Device:LED
- added R15, R16, R17: 500, LED_SMD:LED_0603_1608Metric_Pad1.05x0.95mm_HandSolder, symbol Device:R_Small
- added U1, U2, U5: MAX3077E, Package_SO:SOIC-8_3.9x4.9mm_P1.27mm, symbol MRDT_ICs:MAX3077E
- C1, C2: value .1uF -> 10u
- C3: value 10uF -> 10u
Connections:
- net labels added: +3V3, A1, A2, A3, B1, B2, B3, RX_1, RX_2, RX_3, TX_1, TX_2, TX_3, Y1, Y2, Y3, Z1, Z2, Z3
- net labels removed: +5V, RX_1_IC, RX_1_SL, RX_2_IC, RX_2_SL, RX_3_IC, RX_3_SL, TX_1_IC, TX_1_SL, TX_2_IC, TX_2_SL, TX_3_IC, TX_3_SL
- wire segments 149 -> 185
Other:
- moved on the sheet: C7, C8, Conn1A, Conn1B, Conn2, Conn3, Conn4, D2, D3, D4, D5, D6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

Commit message: Finished BOM
Parts:
- R10, R11, R12, R13, R14, R8, R9: value 10K -> 500
Changed lines of the file:
@@
 P 9650 4100
 F 0 "R8" V 9650 4100 50  0000 C CNN
-F 1 "10K" V 9550 4100 50  0000 C CNN
+F 1 "500" V 9550 4100 50  0000 C CNN
 F 2 "Resistor_SMD:R_0603_1608Metric_Pad1.05x0.95mm_HandSolder" V 9580 4100 50  0001 C CNN
 F 3 "~" H 9650 4100 50  0001 C CNN
@@
 P 9700 4500
 F 0 "R9" V 9700 4500 50  0000 C CNN
-F 1 "10K" V 9600 4500 50  0000 C CNN
+F 1 "500" V 9600 4500 50  0000 C CNN
 F 2 "Resistor_SMD:R_0603_1608Metric_Pad1.05x0.95mm_HandSolder" V 9630 4500 50  0001 C CNN
 F 3 "~" H 9700 4500 50  0001 C CNN
@@
 P 9700 4900
 F 0 "R10" V 9700 4900 50  0000 C CNN
-F 1 "10K" V 9600 4900 50  0000 C CNN
+F 1 "500" V 9600 4900 50  0000 C CNN
 F 2 "Resistor_SMD:R_0603_1608Metric_Pad1.05x0.95mm_HandSolder" V 9630 4900 50  0001 C CNN
 F 3 "~" H 9700 4900 50  0001 C CNN
@@
 P 9700 5300
 F 0 "R11" V 9700 5300 50  0000 C CNN
-F 1 "10K" V 9600 5300 50  0000 C CNN
+F 1 "500" V 9600 5300 50  0000 C CNN
 F 2 "Resistor_SMD:R_0603_1608Metric_Pad1.05x0.95mm_HandSolder" V 9630 5300 50  0001 C CNN
 F 3 "~" H 9700 5300 50  0001 C CNN
@@
 P 9700 5700
 F 0 "R12" V 9700 5700 50  0000 C CNN
-F 1 "10K" V 9600 5700 50  0000 C CNN
+F 1 "500" V 9600 5700 50  0000 C CNN
 F 2 "Resistor_SMD:R_0603_1608Metric_Pad1.05x0.95mm_HandSolder" V 9630 5700 50  0001 C CNN
 F 3 "~" H 9700 5700 50  0001 C CNN
@@
 P 9950 6050
 F 0 "R13" V 9950 6050 50  0000 C CNN
-F 1 "10K" V 9850 6050 50  0000 C CNN
+F 1 "500" V 9850 6050 50  0000 C CNN
 F 2 "Resistor_SMD:R_0603_1608Metric_Pad1.05x0.95mm_HandSolder" V 9880 6050 50  0001 C CNN
 F 3 "~" H 9950 6050 50  0001 C CNN
@@
 P 9950 6350
 F 0 "R14" V 9950 6350 50  0000 C CNN
-F 1 "10K" V 9850 6350 50  0000 C CNN
+F 1 "500" V 9850 6350 50  0000 C CNN
 F 2 "Resistor_SMD:R_0603_1608Metric_Pad1.05x0.95mm_HandSolder" V 9880 6350 50  0001 C CNN
 F 3 "~" H 9950 6350 50  0001 C CNN

Commit message: board review
Parts:
- added R18, R19, R20: 120, Resistor_SMD:R_0603_1608Metric_Pad1.05x0.95mm_HandSolder, symbol Device:R_Small
- C1, C2, C3: value 10u -> .1uF
Connections:
- net A1: now also R18.1
- net A2: now also R19.1
- net A3: now also R20.1
- net B1: now also R18.2
- net B2: now also R19.2
- net B3: now also R20.2
- net M1_SW renamed LF_SW
- net M2_SW renamed LM_SW
- net M3_SW renamed LR_SW
- net M4_SW renamed RF_SW
- net M5_SW renamed RM_SW
- net M6_SW renamed RR_SW
Other:
- note added: "Front Motors"
- note added: "Middle Motors"
- note added: "Rear Motors"
- note removed: "Motor 1,2"
- note removed: "Motor 3,4"
- note removed: "Motor 5,6"
- moved on the sheet: D1, D10, D3, D4, D5, D9, R15, R16, R17, R2, R3, R4
