File: DriveBoard_Hardware/DriveBoard_Hardware.kicad_pcb (KiCad board)
At the start: 2 copper layers, 61 x 93.6 mm, 60 parts, among them SW1 SW_Push, SW2 SW_Push, SW3 SW_Push, SW4 SW_Push, SW5 SW_Push, SW6 SW_Push, SW7 SW_SPDT, U1 MAX3077E, U2 MAX3077E, U3 OKI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

Commit message: board review
Parts:
- added G***: LOGO, MRDT_Silkscreens:0_MRDT_Retro_Logo_34mmX21.5mm, B.Cu at (114.3, 93.0)
- added G***: LOGO, MRDT_Silkscreens:0_MRDT_Logo_20mm, F.Cu at (119.4, 149.6)
- added R18: 120, Resistor_SMD:R_0603_1608Metric_Pad1.05x0.95mm_HandSolder, F.Cu at (77.1, 86.9)
- added R19: 120, Resistor_SMD:R_0603_1608Metric_Pad1.05x0.95mm_HandSolder, F.Cu at (94.9, 86.9)
- added R20: 120, Resistor_SMD:R_0603_1608Metric_Pad1.05x0.95mm_HandSolder, F.Cu at (112.6, 86.9)
- C1, C2, C3: value 10u -> .1uF
- R10, R11, R12, R13, R14, R8, R9: value 10K -> 500
- moved G*** 65.3 mm to (125.5, 89.7)
- moved R14 1.02 mm to (128.1, 99.8)
- moved D17 1.02 mm to (123.8, 99.8)
Connections:
- net M1_SW renamed LF_SW
- net M2_SW renamed LM_SW
- net M3_SW renamed LR_SW
- net M4_SW renamed RF_SW
- net M5_SW renamed RM_SW
- net M6_SW renamed RR_SW
Routing:
- net B3: track 8.25 -> 9.41 mm
- net B2: track 8.25 -> 9.41 mm
- net +3V3: track 196.4 -> 195.2 mm
- net Rspeed: track 21.8 -> 22.4 mm
