File: DriveBoard2020/DriveBoard2020.sch (KiCad schematic (older format))
At the start: 53 parts, among them SW1 SW_DPST_x2, SW2 SW_Push_Dual_x2, SW3 SW_Push_Dual_x2, SW4 SW_Push_Dual_x2, U1 MAX232, U2 MAX232, U3 OKI, U4 TM4C129E_Launchpad, U5 MAX232, U6 OKI

Commit message: started layout
Parts:
- removed SW1: SW_DPST_x2, Button_Switch_THT:SW_CuK_OS102011MA1QN1_SPDT_Angled, symbol Switch:SW_DPST_x2
- removed SW2, SW3, SW4: SW_Push_Dual_x2, Button_Switch_SMD:SW_SPST_TL3305A, symbol Switch:SW_Push_Dual_x2
- added SW0: SW_SPST, Button_Switch_THT:SW_CuK_OS102011MA1QN1_SPDT_Angled, symbol Switch:SW_SPST
- added SW1, SW2, SW3, SW4, SW5, SW6: SW_Push, Button_Switch_SMD:SW_SPST_TL3305A, symbol Switch:SW_Push
- Conn1: symbol MRDT_Connectors:AndersonPP -> DriveBoard2020-rescue:AndersonPP-MRDT_Connectors
- Conn2, Conn3, Conn4, Conn5, Conn6, Conn7: footprint MRDT_Connectors:MOLEX_SL_05_Horizontal -> MRDT_Connectors:MOLEX_SL_05_Vertical; symbol MRDT_Connectors:Molex_SL_05 -> DriveBoard2020-rescue:Molex_SL_05-MRDT_Connectors
- U3, U6: symbol MRDT_Devices:OKI -> DriveBoard2020-rescue:OKI-MRDT_Devices
- U4: symbol MRDT_Shields:TM4C129E_Launchpad -> DriveBoard2020-rescue:TM4C129E_Launchpad-MRDT_Shields
Connections:
- net +3V3: now also SW0.1 (A), SW1.1, SW2.1, SW3.1, SW4.1, SW5.1, SW6.1
- net FL_Motor: now also SW1.2
- net FR_Motor: now also SW2.2
- net ML_Motor: now also SW3.2
- net MR_Motor: now also SW4.2
- net RL_Motor: now also SW5.2
- net RR_Motor: now also SW6.2
- net switch_direction: now also SW0.2 (B)
Changed lines of the file:
@@
 $EndDescr
 $Comp
-L MRDT_Connectors:AndersonPP Conn1
+L DriveBoard2020-rescue:AndersonPP-MRDT_Connectors Conn1
 U 1 1 5D9156E9
 P 750 1550
@@
 $EndComp
 $Comp
-L MRDT_Devices:OKI U3
+L DriveBoard2020-rescue:OKI-MRDT_Devices U3
 U 1 1 5D91F370
 P 2250 1100
@@
 	2450 1450 3000 1450
 $Comp
-L MRDT_Shields:TM4C129E_Launchpad U4
+L DriveBoard2020-rescue:TM4C129E_Launchpad-MRDT_Shields U4
 U 5 1 5D99E152
 P 3650 7000
@@
 $EndComp
 $Comp
-L MRDT_Shields:TM4C129E_Launchpad U4
+L DriveBoard2020-rescue:TM4C129E_Launchpad-MRDT_Shields U4
 U 6 1 5D9A42ED
 P 4250 7000
@@
 Level Shifters
 $Comp
-L MRDT_Connectors:AndersonPP Conn1
+L DriveBoard2020-rescue:AndersonPP-MRDT_Connectors Conn1
 U 2 1 5D9F5218
 P 750 1100
@@
 $EndComp
 $Comp
-L MRDT_Connectors:Molex_SL_05 Conn3
+L DriveBoard2020-rescue:Molex_SL_05-MRDT_Connectors Conn3
 U 1 1 5D9F0837
 P 10000 2350
 F 0 "Conn3" H 9550 2950 60  0000 L CNN
 F 1 "Molex_SL_05" H 9550 3050 60  0000 L CNN
-F 2 "MRDT_Connectors:MOLEX_SL_05_Horizontal" H 10000 2350 60  0001 C CNN
+F 2 "MRDT_Connectors:MOLEX_SL_05_Vertical" H 10000 2350 60  0001 C CNN
 F 3 "" H 10000 2350 60  0001 C CNN
 	1    10000 2350
@@
 $EndComp
 $Comp
-L MRDT_Connectors:Molex_SL_05 Conn4
+L DriveBoard2020-rescue:Molex_SL_05-MRDT_Connectors Conn4
 U 1 1 5D9F0E09
 P 10000 3250
 F 0 "Conn4" H 9400 2850 60  0000 L CNN
 F 1 "Molex_SL_05" H 9400 2950 60  0000 L CNN
-F 2 "MRDT_Connectors:MOLEX_SL_05_Horizontal" H 10000 3250 60  0001 C CNN
+F 2 "MRDT_Connectors:MOLEX_SL_05_Vertical" H 10000 3250 60  0001 C CNN
 F 3 "" H 10000 3250 60  0001 C CNN
 	1    10000 3250
@@
 R3_In
 $Comp
-L MRDT_Connectors:Molex_SL_05 Conn6
+L DriveBoard2020-rescue:Molex_SL_05-MRDT_Connectors Conn6
 U 1 1 5DA4491F
 P 10200 2350
 F 0 "Conn6" H 10200 2300 60  0000 C CNN
 F 1 "Molex_SL_05" H 10300 2200 60  0000 C CNN
-F 2 "MRDT_Connectors:MOLEX_SL_05_Horizontal" H 10200 2350 60  0001 C CNN
+F 2 "MRDT_Connectors:MOLEX_SL_05_Vertical" H 10200 2350 60  0001 C CNN
 F 3 "" H 10200 2350 60  0001 C CNN
 	1    10200 2350
@@
 $EndComp
 $Comp
-L MRDT_Connectors:Molex_SL_05 Conn7
+L DriveBoard2020-rescue:Molex_SL_05-MRDT_Connectors Conn7
 U 1 1 5DA45098
 P 10200 3250
 F 0 "Conn7" H 9800 3000 60  0000 C CNN
 F 1 "Molex_SL_05" H 9950 3100 60  0000 C CNN
-F 2 "MRDT_Connectors:MOLEX_SL_05_Horizontal" H 10200 3250 60  0001 C CNN
+F 2 "MRDT_Connectors:MOLEX_SL_05_Vertical" H 10200 3250 60  0001 C CNN
 F 3 "" H 10200 3250 60  0001 C CNN
 	1    10200 3250
@@
 $EndComp
 $Comp
-L MRDT_Connectors:Molex_SL_05 Conn5
+L DriveBoard2020-rescue:Molex_SL_05-MRDT_Connectors Conn5
 U 1 1 5DA43D44
 P 10200 1500
 F 0 "Conn5" H 9750 2050 60  0000 C CNN
 F 1 "Molex_SL_05" H 9800 2150 60  0000 C CNN
-F 2 "MRDT_Connectors:MOLEX_SL_05_Horizontal" H 10200 1500 60  0001 C CNN
+F 2 "MRDT_Connectors:MOLEX_SL_05_Vertical" H 10200 1500 60  0001 C CNN
 F 3 "" H 10200 1500 60  0001 C CNN
 	1    10200 1500
@@
 Connectors
 $Comp
-L MRDT_Connectors:Molex_SL_05 Conn2
+L DriveBoard2020-rescue:Molex_SL_05-MRDT_Connectors Conn2
 U 1 1 5D9EFF87
 P 10000 1500
 F 0 "Conn2" H 9250 2050 60  0000 L CNN
 F 1 "Molex_SL_05" H 9250 2150 60  0000 L CNN
-F 2 "MRDT_Connectors:MOLEX_SL_05_Horizontal" H 10000 1500 60  0001 C CNN
+F 2 "MRDT_Connectors:MOLEX_SL_05_Vertical" H 10000 1500 60  0001 C CNN
 F 3 "" H 10000 1500 60  0001 C CNN
 	1    10000 1500
@@
 Switches/Buttons
 $Comp
-L Switch:SW_DPST_x2 SW1
-U 1 1 5DAF057E
-P 6350 3400
-F 0 "SW1" H 6350 3635 50  0000 C CNN
-F 1 "SW_DPST_x2" H 6350 3544 50  0000 C CNN
-F 2 "Button_Switch_THT:SW_CuK_OS102011MA1QN1_SPDT_Angled" H 6350 3400 50  0001 C CNN
-F 3 "~" H 6350 3400 50  0001 C CNN
-	1    6350 3400
-	1    0    0    -1
-$EndComp
-$Comp
 L power:+3.3V #PWR0125
 U 1 1 5DAF226A
@@
 	1    0    0    -1
 $EndComp
-Wire Wire Line
-	5700 3400 6150 3400
-Wire Wire Line
-	6550 3400 6700 3400
 Text GLabel 6800 3400 2    39   Output ~ 0
 switch_direction
-$Comp
-L Switch:SW_Push_Dual_x2 SW2
-U 1 1 5DAFC00F
-P 6350 3800
-F 0 "SW2" H 6350 4085 50  0000 C CNN
-F 1 "SW_Push_Dual_x2" H 6350 3994 50  0000 C CNN
-F 2 "Button_Switch_SMD:SW_SPST_TL3305A" H 6350 4000 50  0001 C CNN
-F 3 "~" H 6350 4000 50  0001 C CNN
-	1    6350 3800
-	1    0    0    -1
-$EndComp
 $Comp
 L power:+3.3V #PWR0126
@@
 	1    0    0    -1
 $EndComp
-Wire Wire Line
-	5700 3800 6150 3800
-Wire Wire Line
-	6550 3800 6700 3800
 Text GLabel 6800 3800 2    39   Output ~ 0
 FL_Motor
-$Comp
-L Switch:SW_Push_Dual_x2 SW2
-U 2 1 5DB041AC
-P 6350 4150
-F 0 "SW2" H 6350 4435 50  0000 C CNN
-F 1 "SW_Push_Dual_x2" H 6350 4344 50  0000 C CNN
-F 2 "Button_Switch_SMD:SW_SPST_TL3305A" H 6350 4350 50  0001 C CNN
-F 3 "~" H 6350 4350 50  0001 C CNN
-	2    6350 4150
-	1    0    0    -1
-$EndComp
 $Comp
 L power:+3.3V #PWR0127
@@
 FR_Motor
 $Comp
-L Switch:SW_Push_Dual_x2 SW3
-U 1 1 5DB05D3A
-P 6350 4500
-F 0 "SW3" H 6350 4785 50  0000 C CNN
-F 1 "SW_Push_Dual_x2" H 6350 4694 50  0000 C CNN
-F 2 "Button_Switch_SMD:SW_SPST_TL3305A" H 6350 4700 50  0001 C CNN
-F 3 "~" H 6350 4700 50  0001 C CNN
-	1    6350 4500
-	1    0    0    -1
-$EndComp
-$Comp
 L power:+3.3V #PWR0128
 U 1 1 5DB05D40
@@
 ML_Motor
 $Comp
-L Switch:SW_Push_Dual_x2 SW3
-U 2 1 5DB07B8A
-P 6350 4900
-F 0 "SW3" H 6350 5185 50  0000 C CNN
-F 1 "SW_Push_Dual_x2" H 6350 5094 50  0000 C CNN
-F 2 "Button_Switch_SMD:SW_SPST_TL3305A" H 6350 5100 50  0001 C CNN
-F 3 "~" H 6350 5100 50  0001 C CNN
-	2    6350 4900
-	1    0    0    -1
-$EndComp
-$Comp
 L power:+3.3V #PWR0129
 U 1 1 5DB07B90
@@
 MR_Motor
 $Comp
-L Switch:SW_Push_Dual_x2 SW4
-U 1 1 5DB0989B
-P 6350 5250
-F 0 "SW4" H 6350 5535 50  0000 C CNN
-F 1 "SW_Push_Dual_x2" H 6350 5444 50  0000 C CNN
-F 2 "Button_Switch_SMD:SW_SPST_TL3305A" H 6350 5450 50  0001 C CNN
-F 3 "~" H 6350 5450 50  0001 C CNN
-	1    6350 5250
-	1    0    0    -1
-$EndComp
-$Comp
 L power:+3.3V #PWR0130
 U 1 1 5DB098A1
@@
 Text GLabel 6800 5250 2    39   Output ~ 0
 RL_Motor
-$Comp
-L Switch:SW_Push_Dual_x2 SW4
-U 2 1 5DB0B480
-P 6350 5650
-F 0 "SW4" H 6350 5935 50  0000 C CNN
-F 1 "SW_Push_Dual_x2" H 6350 5844 50  0000 C CNN
-F 2 "Button_Switch_SMD:SW_SPST_TL3305A" H 6350 5850 50  0001 C CNN
-F 3 "~" H 6350 5850 50  0001 C CNN
-	2    6350 5650
-	1    0    0    -1
-$EndComp
 $Comp
 L power:+3.3V #PWR0131
@@
 	3400 1000 3800 1000
 $Comp
-L MRDT_Devices:OKI U6
+L DriveBoard2020-rescue:OKI-MRDT_Devices U6
 U 1 1 5DA04040
 P 4000 1100
@@
 Wire Wire Line
 	650  2950 800  2950
+Wire Wire Line
+	6550 3400 6700 3400
+Wire Wire Line
+	5700 3400 6150 3400
+Wire Wire Line
+	6550 3800 6700 3800
+Wire Wire Line
+	5700 3800 6150 3800
+$Comp
+L Switch:SW_Push SW1
+U 1 1 5DA53EB7
+P 6350 3800
+F 0 "SW1" H 6350 4085 50  0000 C CNN
+F 1 "SW_Push" H 6350 3994 50  0000 C CNN
+F 2 "Button_Switch_SMD:SW_SPST_TL3305A" H 6350 4000 50  0001 C CNN
+F 3 "~" H 6350 4000 50  0001 C CNN
+	1    6350 3800
+	1    0    0    -1
+$EndComp
+$Comp
+L Switch:SW_Push SW2
+U 1 1 5DA5B695
+P 6350 4150
+F 0 "SW2" H 6350 4435 50  0000 C CNN
+F 1 "SW_Push" H 6350 4344 50  0000 C CNN
+F 2 "Button_Switch_SMD:SW_SPST_TL3305A" H 6350 4350 50  0001 C CNN
+F 3 "~" H 6350 4350 50  0001 C CNN
+	1    6350 4150
+	1    0    0    -1
+$EndComp
+$Comp
+L Switch:SW_Push SW3
+U 1 1 5DA5B9FD
+P 6350 4500
+F 0 "SW3" H 6350 4785 50  0000 C CNN
+F 1 "SW_Push" H 6350 4694 50  0000 C CNN
+F 2 "Button_Switch_SMD:SW_SPST_TL3305A" H 6350 4700 50  0001 C CNN
+F 3 "~" H 6350 4700 50  0001 C CNN
+	1    6350 4500
+	1    0    0    -1
+$EndComp
+$Comp
+L Switch:SW_Push SW4
+U 1 1 5DA5BE4A
+P 6350 4900
+F 0 "SW4" H 6350 5185 50  0000 C CNN
+F 1 "SW_Push" H 6350 5094 50  0000 C CNN
+F 2 "Button_Switch_SMD:SW_SPST_TL3305A" H 6350 5100 50  0001 C CNN
+F 3 "~" H 6350 5100 50  0001 C CNN
+	1    6350 4900
+	1    0    0    -1
+$EndComp
+$Comp
+L Switch:SW_Push SW5
+U 1 1 5DA5C536
+P 6350 5250
+F 0 "SW5" H 6350 5535 50  0000 C CNN
+F 1 "SW_Push" H 6350 5444 50  0000 C CNN
+F 2 "Button_Switch_SMD:SW_SPST_TL3305A" H 6350 5450 50  0001 C CNN
+F 3 "~" H 6350 5450 50  0001 C CNN
+	1    6350 5250
+	1    0    0    -1
+$EndComp
+$Comp
+L Switch:SW_Push SW6
+U 1 1 5DA5C839
+P 6350 5650
+F 0 "SW6" H 6350 5935 50  0000 C CNN
+F 1 "SW_Push" H 6350 5844 50  0000 C CNN
+F 2 "Button_Switch_SMD:SW_SPST_TL3305A" H 6350 5850 50  0001 C CNN
+F 3 "~" H 6350 5850 50  0001 C CNN
+	1    6350 5650
+	1    0    0    -1
+$EndComp
+$Comp
+L Switch:SW_SPST SW0
+U 1 1 5DA66B86
+P 6350 3400
+F 0 "SW0" H 6350 3635 50  0000 C CNN
+F 1 "SW_SPST" H 6350 3544 50  0000 C CNN
+F 2 "Button_Switch_THT:SW_CuK_OS102011MA1QN1_SPDT_Angled" H 6350 3400 50  0001 C CNN
+F 3 "~" H 6350 3400 50  0001 C CNN
+	1    6350 3400
+	1    0    0    -1
+$EndComp
 $EndSCHEMATC
