File: DriveBoard2020/DriveBoard2020.sch (KiCad schematic (older format))
At the start: 80 parts, among them SW0 SW_SPST, SW1 SW_Push, SW2 SW_Push, SW3 SW_Push, SW4 SW_Push, SW5 SW_Push, SW6 SW_Push, SW7 SW_Push, SW8 SW_Push, SW9 SW_Push, U1 MAX_3232, U10 TM4C129E_Launchpad, U2 MAX_3232, U3 OKI, U4 TM4C129E_Launchpad, U5 MAX_3232, U6 OKI, U7 OKI, U8 LDD-1500L, U9 TM4C129E_Launchpad

Commit message: minor changes to layout
Parts:
- U10, U9: footprint (none) -> MRDT_Shields:TM4C129E_Launchpad_X9_THT_BOTTOM
Connections:
- net FL_Motor: now also U9.PK4 (C2_2); no longer U4.PD4 (A2_5)
- net FR_Motor: now also U9.PK5 (C2_3); no longer U4.PD5 (A2_6)
- net ML_Motor: now also U9.PM0 (C2_4); no longer U4.PQ0 (A2_7)
- net MR_Motor: now also U9.PM1 (C2_5); no longer U4.PP4 (A2_8)
- net RL_Motor: now also U9.PM2 (C2_6); no longer U4.PN5 (A2_9)
- net RR_Motor: now also U9.PH0 (C2_7); no longer U4.PN4 (A2_10)
Other:
- note removed: "SPI MOSI(3)"
Changed lines of the file:
@@
 F 0 "U10" H 5280 5460 60  0000 L CNN
 F 1 "TM4C129E_Launchpad" H 5830 5010 60  0001 L CNN
-F 2 "" H 5230 4310 60  0001 C CNN
+F 2 "MRDT_Shields:TM4C129E_Launchpad_X9_THT_BOTTOM" H 5230 4310 60  0001 C CNN
 F 3 "" H 5230 4310 60  0001 C CNN
 	3    5230 4310
@@
 F 0 "U10" H 5910 5460 60  0000 L CNN
 F 1 "TM4C129E_Launchpad" H 6260 4910 60  0001 L CNN
-F 2 "" H 5860 4310 60  0001 C CNN
+F 2 "MRDT_Shields:TM4C129E_Launchpad_X9_THT_BOTTOM" H 5860 4310 60  0001 C CNN
 F 3 "" H 5860 4310 60  0001 C CNN
 	4    5860 4310
@@
 Wire Wire Line
 	9700 5750 9700 5800
-Text Notes 4980 5160 2    50   ~ 0
-SPI MOSI(3)
 Text Label 9800 5900 0    50   ~ 0
 Headlight_V1+
@@
 Text Notes 2980 6570 2    39   ~ 0
 Serial 6
-Text GLabel 3230 7220 0    39   Input ~ 0
+Text GLabel 5330 7120 0    39   Input ~ 0
 RR_Motor
-Text GLabel 3230 7120 0    39   Input ~ 0
+Text GLabel 5330 7020 0    39   Input ~ 0
 RL_Motor
-Text GLabel 3230 7020 0    39   Input ~ 0
+Text GLabel 5330 6920 0    39   Input ~ 0
 MR_Motor
-Text GLabel 3230 6920 0    39   Input ~ 0
+Text GLabel 5330 6820 0    39   Input ~ 0
 ML_Motor
-Text GLabel 3230 6820 0    39   Input ~ 0
+Text GLabel 5330 6720 0    39   Input ~ 0
 FR_Motor
-Text GLabel 3230 6720 0    39   Input ~ 0
+Text GLabel 5330 6620 0    39   Input ~ 0
 FL_Motor
 Text GLabel 4230 6920 2    39   Input ~ 0
@@
 F 0 "U9" H 3110 6470 60  0000 L CNN
 F 1 "TM4C129E_Launchpad" H 2610 5260 60  0000 L CNN
-F 2 "" H 3230 5320 60  0001 C CNN
+F 2 "MRDT_Shields:TM4C129E_Launchpad_X9_THT_BOTTOM" H 3230 5320 60  0001 C CNN
 F 3 "" H 3230 5320 60  0001 C CNN
 	1    3230 5320
@@
 U 2 1 5DE90FB1
 P 3880 5320
-F 0 "U9" H 3911 6597 60  0000 C CNN
-F 1 "TM4C129E_Launchpad" H 3911 6491 60  0000 C CNN
-F 2 "" H 3880 5320 60  0001 C CNN
+F 0 "U9" H 4040 6560 60  0000 C CNN
+F 1 "TM4C129E_Launchpad" H 3650 6440 60  0000 C CNN
+F 2 "MRDT_Shields:TM4C129E_Launchpad_X9_THT_BOTTOM" H 3880 5320 60  0001 C CNN
 F 3 "" H 3880 5320 60  0001 C CNN
 	2    3880 5320
@@
 P 5530 7470
 F 0 "U9" H 5835 8068 60  0000 L CNN
-F 1 "TM4C129E_Launchpad" H 4830 7270 60  0000 L CNN
-F 2 "" H 5530 7470 60  0001 C CNN
+F 1 "TM4C129E_Launchpad" H 4870 7320 60  0000 L CNN
+F 2 "MRDT_Shields:TM4C129E_Launchpad_X9_THT_BOTTOM" H 5530 7470 60  0001 C CNN
 F 3 "" H 5530 7470 60  0001 C CNN
 	7    5530 7470
@@
 F 0 "U9" H 6261 8747 60  0000 C CNN
 F 1 "TM4C129E_Launchpad" H 6261 8641 60  0000 C CNN
-F 2 "" H 6230 7470 60  0001 C CNN
+F 2 "MRDT_Shields:TM4C129E_Launchpad_X9_THT_BOTTOM" H 6230 7470 60  0001 C CNN
 F 3 "" H 6230 7470 60  0001 C CNN
 	8    6230 7470

Commit message: working on layout
Parts:
- U4: renamed from U10; footprint MRDT_Shields:TM4C129E_Launchpad_X9_THT_BOTTOM -> MRDT_Shields:TM4C129E_Launchpad_FULL_THT_BOTTOM
- U4: renamed from U9; footprint MRDT_Shields:TM4C129E_Launchpad_X9_THT_BOTTOM -> MRDT_Shields:TM4C129E_Launchpad_FULL_THT_BOTTOM
Connections:
- net FL_Motor: now also U4.PK5 (C2_3); no longer U4.PK4 (C2_2)
- net FR_Motor: now also U4.PM0 (C2_4); no longer U4.PK5 (C2_3)
- net ML_Motor: now also U4.PH1 (C2_8); no longer U4.PM0 (C2_4)
- net MR_Motor: now also U4.PK6 (C2_9); no longer U4.PM1 (C2_5)
- net RL_Motor: now also U4.PQ1 (D2_9); no longer U4.PM2 (C2_6)
- net RR_Motor: now also U4.PP3 (D2_8); no longer U4.PH0 (C2_7)
- net switch_direction: now also U4.PM6 (D2_10); no longer U4.PK2 (B2_7)
Changed lines of the file:
@@
 $EndDescr
 $Comp
-L MRDT_Shields:TM4C129E_Launchpad U10
+L MRDT_Shields:TM4C129E_Launchpad U4
 U 3 1 5BCE44EF
 P 5230 4310
-F 0 "U10" H 5280 5460 60  0000 L CNN
+F 0 "U4" H 5280 5460 60  0000 L CNN
 F 1 "TM4C129E_Launchpad" H 5830 5010 60  0001 L CNN
-F 2 "MRDT_Shields:TM4C129E_Launchpad_X9_THT_BOTTOM" H 5230 4310 60  0001 C CNN
+F 2 "MRDT_Shields:TM4C129E_Launchpad_FULL_THT_BOTTOM" H 5230 4310 60  0001 C CNN
 F 3 "" H 5230 4310 60  0001 C CNN
 	3    5230 4310
@@
 Dout_NeoPixel
 $Comp
-L MRDT_Shields:TM4C129E_Launchpad U10
+L MRDT_Shields:TM4C129E_Launchpad U4
 U 4 1 5BCE45EC
 P 5860 4310
-F 0 "U10" H 5910 5460 60  0000 L CNN
+F 0 "U4" H 5910 5460 60  0000 L CNN
 F 1 "TM4C129E_Launchpad" H 6260 4910 60  0001 L CNN
-F 2 "MRDT_Shields:TM4C129E_Launchpad_X9_THT_BOTTOM" H 5860 4310 60  0001 C CNN
+F 2 "MRDT_Shields:TM4C129E_Launchpad_FULL_THT_BOTTOM" H 5860 4310 60  0001 C CNN
 F 3 "" H 5860 4310 60  0001 C CNN
 	4    5860 4310
@@
 Text Notes 2980 6570 2    39   ~ 0
 Serial 6
-Text GLabel 5330 7120 0    39   Input ~ 0
+Text GLabel 6430 7220 2    39   Input ~ 0
 RR_Motor
-Text GLabel 5330 7020 0    39   Input ~ 0
+Text GLabel 6430 7320 2    39   Input ~ 0
 RL_Motor
-Text GLabel 5330 6920 0    39   Input ~ 0
+Text GLabel 5330 7320 0    39   Input ~ 0
 MR_Motor
+Text GLabel 5330 7220 0    39   Input ~ 0
+ML_Motor
 Text GLabel 5330 6820 0    39   Input ~ 0
-ML_Motor
+FR_Motor
 Text GLabel 5330 6720 0    39   Input ~ 0
-FR_Motor
-Text GLabel 5330 6620 0    39   Input ~ 0
 FL_Motor
-Text GLabel 4230 6920 2    39   Input ~ 0
+Text GLabel 6430 7420 2    39   Input ~ 0
 switch_direction
 $Comp
@@
 	9800 5900 10250 5900
 $Comp
-L MRDT_Shields:TM4C129E_Launchpad U9
+L MRDT_Shields:TM4C129E_Launchpad U4
 U 1 1 5DE8D46B
 P 3230 5320
-F 0 "U9" H 3110 6470 60  0000 L CNN
+F 0 "U4" H 3110 6470 60  0000 L CNN
 F 1 "TM4C129E_Launchpad" H 2610 5260 60  0000 L CNN
-F 2 "MRDT_Shields:TM4C129E_Launchpad_X9_THT_BOTTOM" H 3230 5320 60  0001 C CNN
+F 2 "MRDT_Shields:TM4C129E_Launchpad_FULL_THT_BOTTOM" H 3230 5320 60  0001 C CNN
 F 3 "" H 3230 5320 60  0001 C CNN
 	1    3230 5320
@@
 $EndComp
 $Comp
-L MRDT_Shields:TM4C129E_Launchpad U9
+L MRDT_Shields:TM4C129E_Launchpad U4
 U 2 1 5DE90FB1
 P 3880 5320
-F 0 "U9" H 4040 6560 60  0000 C CNN
+F 0 "U4" H 4040 6560 60  0000 C CNN
 F 1 "TM4C129E_Launchpad" H 3650 6440 60  0000 C CNN
-F 2 "MRDT_Shields:TM4C129E_Launchpad_X9_THT_BOTTOM" H 3880 5320 60  0001 C CNN
+F 2 "MRDT_Shields:TM4C129E_Launchpad_FULL_THT_BOTTOM" H 3880 5320 60  0001 C CNN
 F 3 "" H 3880 5320 60  0001 C CNN
 	2    3880 5320
@@
 $EndComp
 $Comp
-L MRDT_Shields:TM4C129E_Launchpad U9
+L MRDT_Shields:TM4C129E_Launchpad U4
 U 7 1 5DEDC9C8
 P 5530 7470
-F 0 "U9" H 5835 8068 60  0000 L CNN
+F 0 "U4" H 5835 8068 60  0000 L CNN
 F 1 "TM4C129E_Launchpad" H 4870 7320 60  0000 L CNN
-F 2 "MRDT_Shields:TM4C129E_Launchpad_X9_THT_BOTTOM" H 5530 7470 60  0001 C CNN
+F 2 "MRDT_Shields:TM4C129E_Launchpad_FULL_THT_BOTTOM" H 5530 7470 60  0001 C CNN
 F 3 "" H 5530 7470 60  0001 C CNN
 	7    5530 7470
@@
 $EndComp
 $Comp
-L MRDT_Shields:TM4C129E_Launchpad U9
+L MRDT_Shields:TM4C129E_Launchpad U4
 U 8 1 5DEDFAF8
 P 6230 7470
-F 0 "U9" H 6261 8747 60  0000 C CNN
+F 0 "U4" H 6261 8747 60  0000 C CNN
 F 1 "TM4C129E_Launchpad" H 6261 8641 60  0000 C CNN
-F 2 "MRDT_Shields:TM4C129E_Launchpad_X9_THT_BOTTOM" H 6230 7470 60  0001 C CNN
+F 2 "MRDT_Shields:TM4C129E_Launchpad_FULL_THT_BOTTOM" H 6230 7470 60  0001 C CNN
 F 3 "" H 6230 7470 60  0001 C CNN
 	8    6230 7470
