File: Hardware/DriveBoard_2021/DriveBoard_2021.kicad_pcb (KiCad board)
At the start: 2 copper layers, 124.5 x 101.6 mm, 85 parts, among them U1 OKI 3V3, U2 OKI 5V, U3 TM4C129E_Launchpad

Commit message: Changed Top plane to GND and routed 3V3 traces.
Should fix GND islands.
Parts:
- renumbered FL_DRIVE to SW1, FR_DRIVE to SW2, BL_DRIVE to SW3, BR_DRIVE to SW4, LT_TURN to SW5, RT_TURN to SW6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
Connections:
- U3 pad +3V3: Net-(U3-Pad+3V3) -> +3V3
Routing:
- net +3V3: track 92.6 -> 322.6 mm, vias 11 -> 8
- added copper zone on F.Cu, net GND
- removed copper zone on F.Cu, net +3V3
