File: Hardware/DriveBoard_Rev2/DriveBoard_Rev2.kicad_pcb (KiCad board)
At the start: 2 copper layers, 203.2 x 101.9 mm, 62 parts, among them J2 RJ45_LED_Shielded, Q1 Q_NMOS_GDS, Q2 Q_NMOS_GDS, Q3 Q_NMOS_GDS, Q4 Q_NMOS_GDS, Q5 Q_NMOS_GDS, Q6 Q_NMOS_GDS, Q7 Q_NMOS_GDS, Q8 Q_NMOS_GDS, Q9 Q_NMOS_GDS, U1 Teensy4.1_DEV-16771, U2 TSR_1-2450, U3 OKI

Commit message: PCB Layout
Finished PCB Layout
Parts:
- added D1: BLUE, LED_SMD:LED_0603_1608Metric_Pad1.05x0.95mm_HandSolder, F.Cu at (225.6, 62.5)
- added D10: BLUE, LED_SMD:LED_0603_1608Metric_Pad1.05x0.95mm_HandSolder, F.Cu at (238.3, 121.9)
- added D11: BLUE, LED_SMD:LED_0603_1608Metric_Pad1.05x0.95mm_HandSolder, F.Cu at (251.1, 62.5)
- added D12: BLUE, LED_SMD:LED_0603_1608Metric_Pad1.05x0.95mm_HandSolder, F.Cu at (251.0, 75.7)
- added D13: BLUE, LED_SMD:LED_0603_1608Metric_Pad1.05x0.95mm_HandSolder, F.Cu at (251.0, 96.5)
- added D14: BLUE, LED_SMD:LED_0603_1608Metric_Pad1.05x0.95mm_HandSolder, F.Cu at (251.1, 109.3)
- added D15: BLUE, LED_SMD:LED_0603_1608Metric_Pad1.05x0.95mm_HandSolder, F.Cu at (251.0, 121.9)
- added D16: BLUE, LED_SMD:LED_0603_1608Metric_Pad1.05x0.95mm_HandSolder, F.Cu at (241.8, 44.2)
- added D2: BLUE, LED_SMD:LED_0603_1608Metric_Pad1.05x0.95mm_HandSolder, F.Cu at (225.6, 75.7)
- added D3: BLUE, LED_SMD:LED_0603_1608Metric_Pad1.05x0.95mm_HandSolder, F.Cu at (225.7, 96.5)
- added D4: BLUE, LED_SMD:LED_0603_1608Metric_Pad1.05x0.95mm_HandSolder, F.Cu at (225.6, 109.3)
- added D5: BLUE, LED_SMD:LED_0603_1608Metric_Pad1.05x0.95mm_HandSolder, F.Cu at (225.7, 121.9)
- added D6: BLUE, LED_SMD:LED_0603_1608Metric_Pad1.05x0.95mm_HandSolder, F.Cu at (238.3, 62.5)
- added D7: BLUE, LED_SMD:LED_0603_1608Metric_Pad1.05x0.95mm_HandSolder, F.Cu at (238.3, 75.7)
- added D8: BLUE, LED_SMD:LED_0603_1608Metric_Pad1.05x0.95mm_HandSolder, F.Cu at (238.3, 96.5)
- added D9: BLUE, LED_SMD:LED_0603_1608Metric_Pad1.05x0.95mm_HandSolder, F.Cu at (238.3, 109.3)
- added R1: 4.7k, Resistor_SMD:R_0603_1608Metric_Pad0.98x0.95mm_HandSolder, F.Cu at (229.6, 62.5)
- added R10: 120, Resistor_SMD:R_0603_1608Metric_Pad0.98x0.95mm_HandSolder, F.Cu at (221.6, 121.9)
- added R11: 4.7k, Resistor_SMD:R_0603_1608Metric_Pad0.98x0.95mm_HandSolder, F.Cu at (242.3, 62.5)
- added R12: 4.7k, Resistor_SMD:R_0603_1608Metric_Pad0.98x0.95mm_HandSolder, F.Cu at (242.3, 75.7)
- added R13: 4.7k, Resistor_SMD:R_0603_1608Metric_Pad0.98x0.95mm_HandSolder, F.Cu at (242.3, 96.5)
- added R14: 4.7k, Resistor_SMD:R_0603_1608Metric_Pad0.98x0.95mm_HandSolder, F.Cu at (242.4, 109.3)
- added R15: 4.7k, Resistor_SMD:R_0603_1608Metric_Pad0.98x0.95mm_HandSolder, F.Cu at (242.3, 121.9)
- added R16: 120, Resistor_SMD:R_0603_1608Metric_Pad0.98x0.95mm_HandSolder, F.Cu at (234.2, 62.5)
- added R17: 120, Resistor_SMD:R_0603_1608Metric_Pad0.98x0.95mm_HandSolder, F.Cu at (234.2, 75.7)
- added R18: 120, Resistor_SMD:R_0603_1608Metric_Pad0.98x0.95mm_HandSolder, F.Cu at (234.2, 96.5)
- added R19: 120, Resistor_SMD:R_0603_1608Metric_Pad0.98x0.95mm_HandSolder, F.Cu at (234.2, 109.3)
- added R2: 4.7k, Resistor_SMD:R_0603_1608Metric_Pad0.98x0.95mm_HandSolder, F.Cu at (229.6, 75.7)
- added R20: 120, Resistor_SMD:R_0603_1608Metric_Pad0.98x0.95mm_HandSolder, F.Cu at (234.2, 121.9)
- added R21: 4.7k, Resistor_SMD:R_0603_1608Metric_Pad0.98x0.95mm_HandSolder, F.Cu at (255.1, 62.5)
- added R22: 4.7k, Resistor_SMD:R_0603_1608Metric_Pad0.98x0.95mm_HandSolder, F.Cu at (255.0, 75.7)
- added R23: 4.7k, Resistor_SMD:R_0603_1608Metric_Pad0.98x0.95mm_HandSolder, F.Cu at (255.0, 96.5)
- added R24: 4.7k, Resistor_SMD:R_0603_1608Metric_Pad0.98x0.95mm_HandSolder, F.Cu at (255.0, 109.3)
- added R25: 4.7k, Resistor_SMD:R_0603_1608Metric_Pad0.98x0.95mm_HandSolder, F.Cu at (255.0, 121.9)
- added R26: 120, Resistor_SMD:R_0603_1608Metric_Pad0.98x0.95mm_HandSolder, F.Cu at (247.0, 62.5)
- added R27: 120, Resistor_SMD:R_0603_1608Metric_Pad0.98x0.95mm_HandSolder, F.Cu at (246.9, 75.7)
- added R28: 120, Resistor_SMD:R_0603_1608Metric_Pad0.98x0.95mm_HandSolder, F.Cu at (246.9, 96.5)
- added R29: 120, Resistor_SMD:R_0603_1608Metric_Pad0.98x0.95mm_HandSolder, F.Cu at (247.0, 109.3)
- added R3: 4.7k, Resistor_SMD:R_0603_1608Metric_Pad0.98x0.95mm_HandSolder, F.Cu at (229.6, 96.5)
- added R30: 120, Resistor_SMD:R_0603_1608Metric_Pad0.98x0.95mm_HandSolder, F.Cu at (246.9, 121.9)
- added R31: 120, Resistor_SMD:R_0603_1608Metric_Pad0.98x0.95mm_HandSolder, F.Cu at (241.8, 47.2)
- added R4: 4.7k, Resistor_SMD:R_0603_1608Metric_Pad0.98x0.95mm_HandSolder, F.Cu at (229.6, 109.3)
- added R5: 4.7k, Resistor_SMD:R_0603_1608Metric_Pad0.98x0.95mm_HandSolder, F.Cu at (229.7, 121.9)
- added R6: 120, Resistor_SMD:R_0603_1608Metric_Pad0.98x0.95mm_HandSolder, F.Cu at (221.5, 62.5)
- added R7: 120, Resistor_SMD:R_0603_1608Metric_Pad0.98x0.95mm_HandSolder, F.Cu at (221.5, 75.7)
- added R8: 120, Resistor_SMD:R_0603_1608Metric_Pad0.98x0.95mm_HandSolder, F.Cu at (221.6, 96.5)
- added R9: 120, Resistor_SMD:R_0603_1608Metric_Pad0.98x0.95mm_HandSolder, F.Cu at (221.5, 109.3)
- added SW1: SW_Push, Button_Switch_SMD:SW_SPST_TL3305A, F.Cu at (225.6, 56.9)
- added SW10: SW_Push, Button_Switch_SMD:SW_SPST_TL3305A, F.Cu at (225.6, 103.7)
- added SW11: SW_Push, Button_Switch_SMD:SW_SPST_TL3305A, F.Cu at (238.3, 103.7)
- added SW12: SW_Push, Button_Switch_SMD:SW_SPST_TL3305A, F.Cu at (251.0, 103.7)
- added SW13: SW_Push, Button_Switch_SMD:SW_SPST_TL3305A, F.Cu at (225.6, 116.3)
- added SW14: SW_Push, Button_Switch_SMD:SW_SPST_TL3305A, F.Cu at (238.3, 116.3)
- added SW15: SW_Push, Button_Switch_SMD:SW_SPST_TL3305A, F.Cu at (251.0, 116.3)
- added SW16: SW_SPDT, Button_Switch_THT:SW_Slide_1P2T_CK_OS102011MS2Q, F.Cu at (229.6, 46.0)
- added SW2: SW_Push, Button_Switch_SMD:SW_SPST_TL3305A, F.Cu at (238.3, 56.9)
- added SW3: SW_Push, Button_Switch_SMD:SW_SPST_TL3305A, F.Cu at (251.0, 56.9)
- added SW4: SW_Push, Button_Switch_SMD:SW_SPST_TL3305A, F.Cu at (225.6, 70.1)
- added SW5: SW_Push, Button_Switch_SMD:SW_SPST_TL3305A, F.Cu at (238.3, 70.1)
- added SW6: SW_Push, Button_Switch_SMD:SW_SPST_TL3305A, F.Cu at (251.0, 70.1)
- added SW7: SW_Push, Button_Switch_SMD:SW_SPST_TL3305A, F.Cu at (225.6, 90.9)
- added SW8: SW_Push, Button_Switch_SMD:SW_SPST_TL3305A, F.Cu at (238.3, 90.9)
- added SW9: SW_Push, Button_Switch_SMD:SW_SPST_TL3305A, F.Cu at (251.0, 90.9)
- added U4: 74HC148, Package_SO:SOIC-16_4.55x10.3mm_P1.27mm, F.Cu at (210.8, 63.0)
- added U5: 74HC148, Package_SO:SOIC-16_4.55x10.3mm_P1.27mm, F.Cu at (210.8, 104.6)
- added U6: 74HC00, Package_SO:SO-14_5.3x10.2mm_P1.27mm, F.Cu at (200.2, 84.8)
- added V1: Via, MRDT_Drill_Holes:4_40_Hole_Corner, F.Cu at (252.1, 131.7)
- added V2: Via, MRDT_Drill_Holes:4_40_Hole_Corner, F.Cu at (39.5, 45.8)
- added V3: Via, MRDT_Drill_Holes:4_40_Hole_Corner, F.Cu at (252.1, 45.8)
- added V4: Via, MRDT_Drill_Holes:4_40_Hole_Corner, F.Cu at (39.5, 131.7)
- moved C3 11.4 mm to (66.5, 76.2)
- moved Conn1 4.68 mm to (50.0, 50.0)
- moved J1 1.25 mm to (29.4, 73.5)
- renumbered C5 to C3, C3 to C4, C4 to C5, Conn7 to Conn2, Conn5 to Conn3, Conn6 to Conn4, Conn2 to Conn5, Conn3 to Conn6, Conn4 to Conn7, D32 to D17, D33 to D18, D34 to D19, D8 to D20, D9 to D21, D1 to D22, D2 to D23, D3 to D24, D4 to D25, D5 to D26, D6 to D27, D7 to D28, D10 to D29, D11 to D30, J2 to J1, R15 to R32, R16 to R33, R27 to R34, R28 to R35, R29 to R36, R1 to R37, R2 to R38, R3 to R39, R4 to R40, R5 to R41, R6 to R42, R7 to R43, R17 to R44, R18 to R45, R8 to R46, R9 to R47, R10 to R48, R11 to R49, R12 to R50, R13 to R51, R14 to R52, R19 to R53, R20 to R54
Connections:
- Q1 pad 1: Net-(Q1-Pad1) -> GND
- R46 pad 2: Net-(Q1-Pad1) -> GND
- U1 pad 24: BIT3 -> OUT3
- U1 pad 25: BIT2 -> OUT2
- U1 pad 36: BIT1 -> OUT1
- U1 pad 37: BIT0 -> OUT0
- U1 pad 5: DRIVE_REVERSE -> REVERSE
Routing:
- net +3V3: track 129.0 -> 734.2 mm, vias 5 -> 32
- net REVERSE: track 0.00 -> 293.4 mm, vias 0 -> 3
- net OUT3: track 0.00 -> 199.7 mm, vias 0 -> 5
- net OUT0: track 0.00 -> 174.3 mm, vias 0 -> 3
- net OUT1: track 0.00 -> 163.8 mm, vias 0 -> 5
- net OUT2: track 0.00 -> 163.6 mm, vias 0 -> 3
- net B12: track 0.00 -> 91.9 mm, vias 0 -> 4
- net B15: track 0.00 -> 61.8 mm, vias 0 -> 2
- net B7: track 0.00 -> 58.5 mm, vias 0 -> 2
- net B6: track 0.00 -> 58.5 mm
- net B9: track 0.00 -> 58.0 mm, vias 0 -> 2
- net B3: track 0.00 -> 55.6 mm
- net B14: track 0.00 -> 50.9 mm, vias 0 -> 2
- net B5: track 0.00 -> 47.3 mm
- net B8: track 0.00 -> 44.3 mm, vias 0 -> 2
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Other:
- board size 203.2 x 101.9 mm -> 228.6 x 101.9 mm
- board text added: "BM"
- board text added: "Core Board, Rev2 Mars Rover Design Team Missouri S&T, 2023 Jorge Noriega"
- board text added: "FM"
- board text added: "REVERSE"

Commit message: Added Signature
Parts:
- added G***: LOGO, Signatures:Jorge_Noriega_34mmx15mm, F.Cu at (128.5, 132.0)
- added G***: LOGO, MRDT_Silkscreens:0_MRDT_Logo_30mm, F.Cu at (57.4, 122.7)
Routing:
- net +3V3: track 734.2 -> 722.5 mm

Commit message: Core Board PCB
Finished Core Board PCB
Parts:
- added C6: 22uF, Capacitor_SMD:C_0603_1608Metric_Pad1.08x0.95mm_HandSolder, F.Cu at (75.2, 63.0)
- added C7: 22uF, Capacitor_SMD:C_0603_1608Metric_Pad1.08x0.95mm_HandSolder, F.Cu at (79.8, 49.8)
- added D31: GREEN, LED_SMD:LED_0603_1608Metric_Pad1.05x0.95mm_HandSolder, F.Cu at (83.7, 70.9)
- added R55: 300, Resistor_SMD:R_0603_1608Metric_Pad0.98x0.95mm_HandSolder, F.Cu at (83.7, 67.8)
- added U7: TSR_1-2450, MRDT_Devices:TSR_1-2433, F.Cu at (78.2, 43.9)
- C1, C2: value 10uF -> 22uF
- Conn2: footprint MRDT_Connectors:MOLEX_uF_S_03_Vertical -> MRDT_Connectors:MOLEX_SL_03_Vertical
- Conn3, Conn4, Conn5, Conn6, Conn7: footprint MRDT_Connectors:MOLEX_uF_S_09_Vertical -> MRDT_Connectors:MOLEX_SL_09_Vertical
- Q1, Q2, Q3, Q4, Q5, Q6, Q7, Q8, Q9: value Q_NMOS_GDS -> Q_NMOS_DGS; moved to B.Cu
- R46, R47, R48, R49, R50, R51, R52, R53, R54, U4, U5, U6: moved to B.Cu
- U1: footprint MRDT_Shields:Teensy_4_1 -> MRDT_Shields:Teensy_4_1_Ethernet
- moved D16 135.9 mm to (110.9, 80.6)
- moved R31 134.4 mm to (110.9, 77.5)
- moved R1 123.5 mm to (112.0, 100.3)
- moved R2 123.5 mm to (112.0, 113.5)
- moved D11 123.5 mm to (133.5, 100.3)
- moved D12 123.5 mm to (133.3, 113.5)
- moved D6 123.5 mm to (120.7, 100.3)
- moved D7 123.5 mm to (120.7, 113.5)
- moved R11 123.5 mm to (124.7, 100.3)
- moved R12 123.5 mm to (124.7, 113.5)
- moved R22 123.5 mm to (137.4, 113.5)
- moved R26 123.5 mm to (129.4, 100.3)
- moved R27 123.5 mm to (129.3, 113.5)
- moved R6 123.5 mm to (103.8, 100.3)
- moved R7 123.5 mm to (103.9, 113.5)
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Connections:
- net Net-(J1-Pad1) renamed /TX+
- net Net-(J1-Pad4) renamed /RX+
- Conn2 pad 1: +5V -> +5VA
- Conn3 pad 1: FLTX -> GND
- Conn3 pad 2: GND -> FLTX
- Conn3 pad 4: MLTX -> GND
- Conn3 pad 5: GND -> MLTX
- Conn3 pad 7: BLTX -> GND
- Conn3 pad 8: GND -> BLTX
- Conn4 pad 1: FRTX -> GND
- Conn4 pad 2: GND -> FRTX
- Conn4 pad 4: MRTX -> GND
- Conn4 pad 5: GND -> MRTX
- Conn4 pad 7: BRTX -> GND
- Conn4 pad 8: GND -> BRTX
- Conn5 pad 1: +5V -> GND
- Conn5 pad 2: GND -> +5V
- Conn5 pad 4: +5V -> GND
- Conn5 pad 5: GND -> +5V
- Conn5 pad 7: +5V -> GND
- Conn5 pad 8: GND -> +5V
- Conn6 pad 1: +5V -> GND
- Conn6 pad 2: GND -> +5V
- Conn6 pad 4: +5V -> GND
- Conn6 pad 5: GND -> +5V
- Conn6 pad 7: +5V -> GND
- Conn6 pad 8: GND -> +5V
- Conn7 pad 1: +5V -> GND
- Conn7 pad 2: GND -> +5V
- Conn7 pad 4: +5V -> GND
- Conn7 pad 5: GND -> +5V
- Conn7 pad 7: +5V -> GND
- Conn7 pad 8: GND -> +5V
- D27 pad 2: Net-(D27-Pad2) -> Net-(R42-Pad1)
- D28 pad 2: Net-(D28-Pad2) -> Net-(R43-Pad1)
- D29 pad 2: Net-(D29-Pad2) -> Net-(R44-Pad1)
- D30 pad 2: Net-(D30-Pad2) -> Net-(R45-Pad1)
- J1 pad 3: Net-(J1-Pad3) -> /TX-
- J1 pad 6: Net-(J1-Pad6) -> /RX-
- Q1 pad 2: Net-(D22-Pad1) -> Net-(R46-Pad2)
- Q1 pad 3: GND -> Net-(D22-Pad1)
- Q2 pad 1: Net-(Q2-Pad1) -> GND
- Q2 pad 2: Net-(D23-Pad1) -> Net-(R47-Pad2)
- Q2 pad 3: GND -> Net-(D23-Pad1)
- Q3 pad 1: Net-(Q3-Pad1) -> GND
- Q3 pad 2: Net-(D24-Pad1) -> Net-(R48-Pad2)
- Q3 pad 3: GND -> Net-(D24-Pad1)
- Q4 pad 1: Net-(Q4-Pad1) -> GND
- Q4 pad 2: Net-(D25-Pad1) -> Net-(R49-Pad2)
- Q4 pad 3: GND -> Net-(D25-Pad1)
- Q5 pad 1: Net-(Q5-Pad1) -> GND
- Q5 pad 2: Net-(D26-Pad1) -> Net-(R50-Pad2)
- Q5 pad 3: GND -> Net-(D26-Pad1)
- Q6 pad 1: Net-(Q6-Pad1) -> GND
- Q6 pad 2: Net-(D27-Pad1) -> Net-(R51-Pad2)
- Q6 pad 3: GND -> Net-(D27-Pad1)
- Q7 pad 1: Net-(Q7-Pad1) -> GND
- Q7 pad 2: Net-(D28-Pad1) -> Net-(R52-Pad2)
- Q7 pad 3: GND -> Net-(D28-Pad1)
- Q8 pad 1: Net-(Q8-Pad1) -> GND
- Q8 pad 2: Net-(D29-Pad1) -> Net-(R53-Pad2)
- Q8 pad 3: GND -> Net-(D29-Pad1)
- Q9 pad 1: Net-(Q9-Pad1) -> GND
- Q9 pad 2: Net-(D30-Pad1) -> Net-(R54-Pad2)
- Q9 pad 3: GND -> Net-(D30-Pad1)
- R37 pad 1: +5V -> Net-(D22-Pad2)
- R37 pad 2: Net-(D22-Pad2) -> +5V
- R38 pad 1: +5V -> Net-(D23-Pad2)
- R38 pad 2: Net-(D23-Pad2) -> +5V
- R39 pad 1: +5V -> Net-(D24-Pad2)
- R39 pad 2: Net-(D24-Pad2) -> +5V
- R40 pad 1: +5V -> Net-(D25-Pad2)
- R40 pad 2: Net-(D25-Pad2) -> +5V
- R41 pad 1: +5V -> Net-(D26-Pad2)
- R41 pad 2: Net-(D26-Pad2) -> +5V
- R42 pad 1: +5V -> Net-(R42-Pad1)
- R42 pad 2: Net-(D27-Pad2) -> +5V
- R43 pad 1: +5V -> Net-(R43-Pad1)
- R43 pad 2: Net-(D28-Pad2) -> +5V
- R44 pad 1: +5V -> Net-(R44-Pad1)
- R44 pad 2: Net-(D29-Pad2) -> +5V
- R45 pad 1: +5V -> Net-(R45-Pad1)
- R45 pad 2: Net-(D30-Pad2) -> +5V
- R46 pad 2: GND -> Net-(R46-Pad2)
- R47 pad 2: Net-(Q2-Pad1) -> Net-(R47-Pad2)
- R48 pad 2: Net-(Q3-Pad1) -> Net-(R48-Pad2)
- R49 pad 2: Net-(Q4-Pad1) -> Net-(R49-Pad2)
- R50 pad 2: Net-(Q5-Pad1) -> Net-(R50-Pad2)
- R51 pad 2: Net-(Q6-Pad1) -> Net-(R51-Pad2)
- R52 pad 2: Net-(Q7-Pad1) -> Net-(R52-Pad2)
- R53 pad 2: Net-(Q8-Pad1) -> Net-(R53-Pad2)
- R54 pad 2: Net-(Q9-Pad1) -> Net-(R54-Pad2)
- U1 pad R-: (no net) -> /RX-
- U1 pad T-: (no net) -> /TX-
- U4 pad 10: +3V3 -> +5V
- U4 pad 16: +3V3 -> +5V
- U5 pad 16: +3V3 -> +5V
Routing:
- net +3V3: track 722.5 -> 512.1 mm, vias 32 -> 3
- net REVERSE: track 293.4 -> 138.3 mm, vias 3 -> 2
- net +5V: track 310.8 -> 434.0 mm, vias 11 -> 2
- net FLTX: track 199.7 -> 118.6 mm, vias 3 -> 2
- net ServoPWM7: track 84.1 -> 163.3 mm, vias 4 -> 2
- net MRTX: track 136.3 -> 59.0 mm, vias 3 -> 1
- net OUT0: track 174.3 -> 97.3 mm, vias 3 -> 2
- net OUT3: track 199.7 -> 123.8 mm, vias 5 -> 4
- net FLRX: track 196.6 -> 121.4 mm, vias 3 -> 2
- net FRTX: track 195.0 -> 121.1 mm, vias 3 -> 2
- net MRRX: track 128.4 -> 55.0 mm, vias 3 -> 1
- net OUT1: track 163.8 -> 91.7 mm, vias 5 -> 2
- net BRTX: track 151.1 -> 79.2 mm, vias 3 -> 1
- net OUT2: track 163.6 -> 93.3 mm, vias 3 -> 2
- net FRRX: track 191.6 -> 122.9 mm, vias 3 -> 2
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Other:
- board size 228.6 x 101.9 mm -> 152.4 x 101.9 mm
- board text added: "5VA"
- board text added: "Core Board, Rev1 Mars Rover Design Team Missouri S&T, 2023 Jorge Noriega"
- board text removed: "Core Board, Rev2 Mars Rover Design Team Missouri S&T, 2023 Jorge Noriega"

Commit message: Core Board PCB
Layout Finished
Parts:
- C1, C4, C6: footprint Capacitor_SMD:C_0603_1608Metric_Pad1.08x0.95mm_HandSolder -> Capacitor_THT:CP_Radial_D5.0mm_P2.00mm
- moved D20 5.30 mm to (67.6, 75.7)
- moved R32 5.30 mm to (63.0, 75.7)
- moved R33 5.30 mm to (63.0, 70.6)
- moved D21 5.30 mm to (67.6, 70.6)
- moved R35 4.83 mm to (79.1, 72.6)
- moved R36 4.83 mm to (87.6, 72.6)
- moved R55 4.83 mm to (83.4, 72.6)
- moved R34 4.83 mm to (74.9, 72.6)
- moved D19 4.83 mm to (87.6, 75.7)
- moved D31 4.83 mm to (83.4, 75.7)
- moved D17 4.83 mm to (74.9, 75.7)
- moved D18 4.83 mm to (79.2, 75.7)
- moved C6 4.29 mm to (73.7, 67.1)
- moved C2 3.92 mm to (80.8, 66.8), turned to -90 degrees
- moved U2 2.77 mm to (78.2, 59.7)
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Connections:
- U4 pad 10: +5V -> +3V3
- U4 pad 16: +5V -> +3V3
- U5 pad 16: +5V -> +3V3
Routing:
- net +5V: track 434.0 -> 303.2 mm, vias 2 -> 0
- net +3V3: track 512.1 -> 578.5 mm, vias 3 -> 5
- net +36V: track 76.6 -> 85.0 mm
- net LEDTX: track 28.5 -> 25.3 mm
- net LEDRX: track 35.5 -> 32.9 mm
- net +5VA: track 38.4 -> 40.9 mm
- net GND: vias 0 -> 1
Other:
- board size 152.4 x 101.9 mm -> 152.4 x 101.6 mm

Commit message: Final Core Board
Parts:
- moved G*** 0.06 mm to (72.4, 134.1)
