File: Hardware/DriveBoard_Rev2/DriveBoard_Rev2.kicad_sch (KiCad schematic)
At the start: 91 parts, among them J1 6P6C, J2 RJ45_LED_Shielded, Q1 Q_NMOS_GDS, Q2 Q_NMOS_GDS, Q3 Q_NMOS_GDS, Q4 Q_NMOS_GDS, Q5 Q_NMOS_GDS, Q6 Q_NMOS_GDS, Q7 Q_NMOS_GDS, U1 Teensy4.1_DEV-16771, U2 OKI, U3 OKI

Commit message: Schematic Review
Updated connectors, power, notations, pin assignments, and started to construct an Encoder for buttons
Parts:
- removed Conn10, Conn2, Conn5, Conn6, Conn7, Conn8, Conn9: Molex_SL_03, symbol MRDT_Connectors:Molex_SL_03
- removed Conn11: Molex_SL_02, symbol MRDT_Connectors:Molex_SL_02
- removed D10, D11, D12, D13, D14, D15, D16, D17, D18, D19, D8, D9: CDBU40-HF, Diode_SMD:D_0603_1608Metric, symbol Diode:CDBU40-HF
- removed D20, D22, D24, D26, D28, D30: YELLOW, symbol Device:LED
- removed D21, D23, D25, D27, D29, D31: BLUE, symbol Device:LED
- removed J1: 6P6C, symbol Connector:6P6C
- removed R15, R16, R17, R18, R19, R20, R21, R22, R23, R24, R25, R26: 100, symbol Device:R
- removed U2: OKI, symbol MRDT_Devices:OKI
- added Conn2, Conn? (x2): Molex_SL_09, symbol MRDT_Connectors:Molex_SL_09
- added Conn?: Molex_SL_03, symbol MRDT_Connectors:Molex_SL_03
- added D?: YELLOW, symbol Device:LED
- added D?: BLUE, symbol Device:LED
- added R?: 300, symbol Device:R
- added R?: 100, symbol Device:R
- added U?: TSR_1-2450, Converter_DCDC:Converter_DCDC_TRACO_TSR-1_THT, symbol Regulator_Switching:TSR_1-2450
Connections:
- net +36V: now also U?.1 (Vin)
- net +5V: now also Conn2.1, Conn2.4, Conn2.7, Conn?.1, U?.3 (Vout)
- net BLRX: now also Conn?.9
- net BLTX: now also Conn?.7
- net BRRX: now also Conn?.9
- net BRTX: now also Conn?.7
- net FLRX: now also Conn?.3
- net FLTX: now also Conn?.1
- net FRRX: now also Conn?.3
- net FRTX: now also Conn?.1
- net GND: now also C5.1, J2.8, J2.9, Conn2.2, Conn2.5, Conn2.8, Conn?.2, Conn?.2, Conn?.2, Conn?.5, Conn?.5, Conn?.8, Conn?.8, D?.1 (K), D?.1 (K), U?.2 (GND)
- net MLRX: now also Conn?.6
- net MLTX: now also Conn?.4
- net MRRX: now also Conn?.6
- net MRTX: now also Conn?.4
- net NeoPixels: now also Conn?.3
- net ServoPWM1: now also Conn2.9; no longer Conn3.9
- net ServoPWM2: now also Conn2.6; no longer Conn3.6
- net ServoPWM3: now also Conn2.3; no longer Conn3.3
- net ServoPWM4: now also Conn3.9; no longer Conn4.9
- net ServoPWM5: now also Conn3.6; no longer Conn4.6
- net ServoPWM6: now also Conn3.3; no longer Conn4.3
- net ServoPWM7: now also Conn4.9, U1.18 (A4); no longer U1.5 (IN2)
- net at J2.1: now also U1.T+
- net at J2.10: now also U1.LED
- net at J2.2, J2.5: now also C5.2; no longer C5.1
- net at J2.3: now also U1.T (T-)
- net at J2.4: now also U1.R+
- net at J2.6: now also U1.R (R-)
- net ServoPWM9: now reaches U1.12 (MISO)
- net ServoPWM9: now also Conn4.3
- net ServoPWM8: now reaches U1.19 (A5)
- net ServoPWM8: now also Conn4.6
- net LEDTX: now reaches U1.22 (A8)
- net LEDTX: now also R?.1
- net LEDRX: now reaches U1.23 (A9)
- net LEDRX: now also R?.1
- net BIT3: now reaches U1.24 (A10)
- net BIT2: now reaches U1.25 (A11)
- net BIT1: now reaches U1.36 (CS2)
- net BIT0: now reaches U1.37 (CS3)
- new net: D?.2 (A), R?.2 (x2)
- new net DRIVE_REVERSE: U1.5 (IN2)
- no-connect marks 38 -> 24
Other:
- note added: "Power LEDs"
- note removed: "Board LEDs"
- moved on the sheet: C5, D1, D2, D3, D32, D33, D34, D4, D5, D6, D7, J2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

Commit message: PCB Layout
Updated the footnotes.
Started and almost finished the layout.
Still needs buttons and encoder.
Parts:
- added D10, D11: BLUE, LED_SMD:LED_0603_1608Metric_Pad1.05x0.95mm_HandSolder, symbol Device:LED
- added Q8, Q9: Q_NMOS_GDS, Package_TO_SOT_SMD:SOT-23, symbol Device:Q_NMOS_GDS
- added R17, R18: 300, Resistor_SMD:R_0603_1608Metric_Pad0.98x0.95mm_HandSolder, symbol Device:R
- added R19, R20: 510, Resistor_SMD:R_0603_1608Metric_Pad0.98x0.95mm_HandSolder, symbol Device:R
- added SW1: SW_Push, Button_Switch_SMD:SW_SPST_TL3305A, symbol Switch:SW_Push
- C1, C2, C3, C4, C5: footprint (none) -> Capacitor_SMD:C_0603_1608Metric_Pad1.08x0.95mm_HandSolder
- Conn1: footprint (none) -> MRDT_Connectors:Square_Anderson_2_H_Side_By_Side
- Conn2, Conn3, Conn4: footprint (none) -> MRDT_Connectors:MOLEX_uF_S_09_Vertical
- Conn5, Conn6: renamed from Conn?; footprint (none) -> MRDT_Connectors:MOLEX_uF_S_09_Vertical
- Conn7: renamed from Conn?; footprint (none) -> MRDT_Connectors:MOLEX_uF_S_03_Vertical
- D1, D2, D3, D32, D33, D34, D4, D5, D6, D7: footprint (none) -> LED_SMD:LED_0603_1608Metric_Pad1.05x0.95mm_HandSolder
- D8, D9: renamed from D?; footprint (none) -> LED_SMD:LED_0603_1608Metric_Pad1.05x0.95mm_HandSolder
- J2: footprint (none) -> MRDT_Connectors:RJ45_Teensy
- Q1, Q2, Q3, Q4, Q5, Q6, Q7: footprint (none) -> Package_TO_SOT_SMD:SOT-23
- R1, R10, R11, R12, R13, R14, R2, R27, R28, R29, R3, R4, R5, R6, R7, R8, R9: footprint (none) -> Resistor_SMD:R_0603_1608Metric_Pad0.98x0.95mm_HandSolder
- R15, R16: renamed from R?; footprint (none) -> Resistor_SMD:R_0603_1608Metric_Pad0.98x0.95mm_HandSolder
- U1: footprint MODULE_DEV-16771 -> MRDT_Shields:Teensy_4_1
- U2: renamed from U?; footprint Converter_DCDC:Converter_DCDC_TRACO_TSR-1_THT -> MRDT_Devices:TSR_1-2433
- U3: footprint (none) -> MRDT_Devices:OKI_Horizontal
Connections:
- net +5V: now also R17.1, R18.1
- net BLRX: now also Conn5.9; no longer Conn6.9
- net BLTX: now also Conn5.7; no longer Conn6.7
- net BRRX: now also Conn6.9; no longer Conn5.9
- net BRTX: now also Conn6.7; no longer Conn5.7
- net FLRX: now also Conn5.3; no longer Conn6.3
- net FLTX: now also Conn5.1; no longer Conn6.1
- net FRRX: now also Conn6.3; no longer Conn5.3
- net FRTX: now also Conn6.1; no longer Conn5.1
- net GND: now also C5.2, Q8.3 (S), Q9.3 (S), SW1.2; no longer C5.1
- net MLRX: now also Conn5.6; no longer Conn6.6
- net MLTX: now also Conn5.4; no longer Conn6.4
- net MRRX: now also Conn6.6; no longer Conn5.6
- net MRTX: now also Conn6.4; no longer Conn5.4
- net ServoPWM8: now also R19.1
- net ServoPWM9: now also R20.1
- net at J2.2, J2.5: now also C5.1; no longer C5.2
- net at Q1.1 (G), R8.2: now also SW1.1
- new net: Q8.1 (G), R19.2
- new net: D11.2 (A), R18.2
- new net: Q9.1 (G), R20.2
- new net: D11.1 (K), Q9.2 (D)
- new net: D10.2 (A), R17.2
- new net: D10.1 (K), Q8.2 (D)
Other:
- moved on the sheet: C5, Conn7, D1, D2, D3, D32, D33, D34, D4, D5, D6, D7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

Commit message: PCB Layout
Finished PCB Layout
Parts:
- added D1, D10, D11, D12, D13, D14, D15, D16, D2, D3, D4, D5, D6, D7, D8, D9: BLUE, LED_SMD:LED_0603_1608Metric_Pad1.05x0.95mm_HandSolder, symbol Device:LED
- added R1, R11, R12, R13, R14, R15, R2, R21, R22, R23, R24, R25, R3, R4, R5: 4.7k, Resistor_SMD:R_0603_1608Metric_Pad0.98x0.95mm_HandSolder, symbol Device:R
- added R10, R16, R17, R18, R19, R20, R26, R27, R28, R29, R30, R31, R6, R7, R8, R9: 120, Resistor_SMD:R_0603_1608Metric_Pad0.98x0.95mm_HandSolder, symbol Device:R
- added SW10, SW11, SW12, SW13, SW14, SW15, SW2, SW3, SW4, SW5, SW6, SW7, SW8, SW9: SW_Push, Button_Switch_SMD:SW_SPST_TL3305A, symbol Switch:SW_Push
- added SW16: SW_SPDT, Button_Switch_THT:SW_Slide_1P2T_CK_OS102011MS2Q, symbol Switch:SW_SPDT
- added U4, U5: 74HC148, Package_SO:SOIC-16_4.55x10.3mm_P1.27mm, symbol 74xx:74LS148
- added U6: 74HC00, Package_SO:SO-14_5.3x10.2mm_P1.27mm, symbol 74xx:74HC00
- added V1, V2, V3, V4: Via, MRDT_Drill_Holes:4_40_Hole_Corner, symbol MRDT_Drill_Holes:Via
- renumbered C5 to C3, C3 to C4, C4 to C5, Conn7 to Conn2, Conn5 to Conn3, Conn6 to Conn4, Conn2 to Conn5, Conn3 to Conn6, Conn4 to Conn7, D32 to D17, D33 to D18, D34 to D19, D8 to D20, D9 to D21, D1 to D22, D2 to D23, D3 to D24, D4 to D25, D5 to D26, D6 to D27, D7 to D28, D10 to D29, D11 to D30, J2 to J1, R15 to R32, R16 to R33, R27 to R34, R28 to R35, R29 to R36, R1 to R37, R2 to R38, R3 to R39, R4 to R40, R5 to R41, R6 to R42, R7 to R43, R17 to R44, R18 to R45, R8 to R46, R9 to R47, R10 to R48, R11 to R49, R12 to R50, R13 to R51, R14 to R52, R19 to R53, R20 to R54
Connections:
- net +3V3: now also D1.2 (A), D10.2 (A), D11.2 (A), D12.2 (A), D13.2 (A), D14.2 (A), D15.2 (A), D2.2 (A), D3.2 (A), D4.2 (A), D5.2 (A), D6.2 (A), D7.2 (A), D8.2 (A), D9.2 (A), R1.1, R11.1, R12.1, R13.1, R14.1, R15.1, R2.1, R21.1, R22.1, R23.1, R24.1, R25.1, R3.1, R4.1, R5.1, SW16.3 (C), U4.10 (IO), U4.16 (VCC), U5.16 (VCC), U6.14 (VCC)
- net GND: now also Q1.1 (G), R46.2, SW1.1, D16.1 (K), SW10.1, SW11.1, SW12.1, SW13.1, SW14.1, SW15.1, SW16.1 (A), SW2.1, SW3.1, SW4.1, SW5.1, SW6.1, SW7.1, SW8.1, SW9.1, U4.8 (GND), U5.5 (EI), U5.8 (GND), U6.7 (GND); no longer SW1.2
- net BIT0 renamed OUT0
- net OUT0: now also U6.3
- net BIT1 renamed OUT1
- net OUT1: now also U6.6
- net BIT2 renamed OUT2
- net OUT2: now also U6.8
- net BIT3 renamed OUT3
- net OUT3: now also U4.5 (EI), U5.15 (EO)
- net DRIVE_REVERSE renamed REVERSE
- net REVERSE: now also R31.2, SW16.2 (B)
- new net: D13.1 (K), R28.2
- new net: D10.1 (K), R20.2
- new net: D11.1 (K), R26.2
- new net: D5.1 (K), R10.2
- new net: D9.1 (K), R19.2
- new net: D2.1 (K), R7.2
- new net: D6.1 (K), R16.2
- new net: D1.1 (K), R6.2
- new net: D8.1 (K), R18.2
- new net: D3.1 (K), R8.2
- new net: U4.7 (S1), U6.4
- new net: U5.7 (S1), U6.5
- new net: D12.1 (K), R27.2
- new net: D16.2 (A), R31.1
- new net: D15.1 (K), R30.2
- new net: D4.1 (K), R9.2
- new net: U4.9 (S0), U6.1
- new net: U5.9 (S0), U6.2
- new net: U4.6 (S2), U6.9
- new net: U5.6 (S2), U6.10
- new net: D7.1 (K), R17.2
- new net: D14.1 (K), R29.2
- new net B1: R1.2, R6.1, SW1.2, U4.11 (I1)
- new net B10: R4.2, R9.1, SW10.2, U5.12 (I2)
- new net B11: R14.2, R19.1, SW11.2, U5.13 (I3)
- new net B12: R24.2, R29.1, SW12.2, U5.1 (I4)
- new net B13: R10.1, R5.2, SW13.2, U5.2 (I5)
- new net B14: R15.2, R20.1, SW14.2, U5.3 (I6)
- new net B15: R25.2, R30.1, SW15.2, U5.4 (I7)
- new net B2: R11.2, R16.1, SW2.2, U4.12 (I2)
- new net B3: R21.2, R26.1, SW3.2, U4.13 (I3)
- new net B4: R2.2, R7.1, SW4.2, U4.1 (I4)
- new net B5: R12.2, R17.1, SW5.2, U4.2 (I5)
- new net B6: R22.2, R27.1, SW6.2, U4.3 (I6)
- new net B7: R3.2, R8.1, SW7.2, U4.4 (I7)
- new net B8: R13.2, R18.1, SW8.2, U5.10 (IO)
- new net B9: R23.2, R28.1, SW9.2, U5.11 (I1)
- no-connect marks 24 -> 30
Other:
- note added: "Buttons"
- note added: "Encoders"
- note added: "Reverse"
- note added: "VIAs"
- moved on the sheet: C3, Conn2, Conn3, Conn4, Conn5, Conn6, Conn7, D17, D18, D19, D20, D21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

Commit message: Core Board PCB
Finished Core Board PCB
Parts:
- removed Q1, Q2, Q3, Q4, Q5, Q6, Q7, Q8, Q9: Q_NMOS_GDS, Package_TO_SOT_SMD:SOT-23, symbol Device:Q_NMOS_GDS
- added C6, C7: 22uF, Capacitor_SMD:C_0603_1608Metric_Pad1.08x0.95mm_HandSolder, symbol Device:C
- added D31: GREEN, LED_SMD:LED_0603_1608Metric_Pad1.05x0.95mm_HandSolder, symbol Device:LED
- added Q1, Q2, Q3, Q4, Q5, Q6, Q7, Q8, Q9: Q_NMOS_DGS, Package_TO_SOT_SMD:SOT-23, symbol Device:Q_NMOS_DGS
- added R55: 300, Resistor_SMD:R_0603_1608Metric_Pad0.98x0.95mm_HandSolder, symbol Device:R
- added U7: TSR_1-2450, MRDT_Devices:TSR_1-2433, symbol Regulator_Switching:TSR_1-2450
- C1, C2: value 10uF -> 22uF
- Conn2: footprint MRDT_Connectors:MOLEX_uF_S_03_Vertical -> MRDT_Connectors:MOLEX_SL_03_Vertical
- Conn3, Conn4, Conn5, Conn6, Conn7: footprint MRDT_Connectors:MOLEX_uF_S_09_Vertical -> MRDT_Connectors:MOLEX_SL_09_Vertical
- U1: footprint MRDT_Shields:Teensy_4_1 -> MRDT_Shields:Teensy_4_1_Ethernet
Connections:
- net +36V: now also C6.2, U7.1 (Vin)
- net +3V3: no longer U4.10 (IO), U4.16 (VCC), U5.16 (VCC)
- net +5V: now also Conn5.2, Conn5.5, Conn5.8, Conn6.2, Conn6.5, Conn6.8, Conn7.2, Conn7.5, Conn7.8, R37.2, R38.2, R39.2, R40.2, R41.2, R42.2, R43.2, R44.2, R45.2, U4.10 (IO), U4.16 (VCC), U5.16 (VCC); no longer Conn2.1, Conn5.1, Conn5.4, Conn5.7, Conn6.1, Conn6.4, Conn6.7, Conn7.1, Conn7.4, Conn7.7, R37.1, R38.1, R39.1, R40.1, R41.1, R42.1, R43.1, R44.1, R45.1
- net BLTX: now also Conn3.8; no longer Conn3.7
- net BRTX: now also Conn4.8; no longer Conn4.7
- net FLTX: now also Conn3.2; no longer Conn3.1
- net FRTX: now also Conn4.2; no longer Conn4.1
- net GND: now also Conn3.1, Conn3.4, Conn3.7, Conn4.1, Conn4.4, Conn4.7, Conn5.1, Conn5.4, Conn5.7, Conn6.1, Conn6.4, Conn6.7, Conn7.1, Conn7.4, Conn7.7, C6.1, C7.1, D31.1 (K), Q1.1 (D), Q2.1 (D), Q3.1 (D), Q4.1 (D), Q5.1 (D), Q6.1 (D), Q7.1 (D), Q8.1 (D), Q9.1 (D), U7.2 (GND); no longer Conn3.2, Conn3.5, Conn3.8, Conn4.2, Conn4.5, Conn4.8, Conn5.2, Conn5.5, Conn5.8, Conn6.2, Conn6.5, Conn6.8, Conn7.2, Conn7.5, Conn7.8, R46.2
- net MLTX: now also Conn3.5; no longer Conn3.4
- net MRTX: now also Conn4.5; no longer Conn4.4
- net at R53.2: now also Q8.2 (G)
- net at R52.2: now also Q7.2 (G)
- net at D28.1 (K): now also Q7.3 (S)
- net at D23.1 (K): now also Q2.3 (S)
- net at D23.2 (A): now also R38.1; no longer R38.2
- net at D25.2 (A): now also R40.1; no longer R40.2
- net at R48.2: now also Q3.2 (G)
- net at D24.1 (K): now also Q3.3 (S)
- net at R47.2: now also Q2.2 (G)
- net at D26.2 (A): now also R41.1; no longer R41.2
- net TX+: now reaches J1.1, U1.T+
- net TX-: now reaches J1.3, U1.T (T-)
- net RX+: now reaches J1.4, U1.R+
- net RX-: now reaches J1.6, U1.R (R-)
- net at D30.2 (A): now also R45.1; no longer R45.2
- net at D22.1 (K): now also Q1.3 (S)
- net at D22.2 (A): now also R37.1; no longer R37.2
- net at R54.2: now also Q9.2 (G)
- net at D30.1 (K): now also Q9.3 (S)
- net at D29.2 (A): now also R44.1; no longer R44.2
- net at R50.2: now also Q5.2 (G)
- net at D26.1 (K): now also Q5.3 (S)
- net at D24.2 (A): now also R39.1; no longer R39.2
- net at R51.2: now also Q6.2 (G)
- net at D27.1 (K): now also Q6.3 (S)
- net at R49.2: now also Q4.2 (G)
- net at D25.1 (K): now also Q4.3 (S)
- net at D27.2 (A): now also R42.1; no longer R42.2
- net at D28.2 (A): now also R43.1; no longer R43.2
- net at D29.1 (K): now also Q8.3 (S)
- new net: Q1.2 (G), R46.2
- new net: D31.2 (A), R55.2
- new net +5VA: C7.2, Conn2.1, R55.1, U7.3 (Vout)
Other:
- moved on the sheet: C4, C5, R37, R38, R39, R40, R41, R42, R43, R44, R45

Commit message: Core Board PCB
Layout Finished
Parts:
- C1, C4, C6: footprint Capacitor_SMD:C_0603_1608Metric_Pad1.08x0.95mm_HandSolder -> Capacitor_THT:CP_Radial_D5.0mm_P2.00mm
Connections:
- net +3V3: now also U4.10 (IO), U4.16 (VCC), U5.16 (VCC)
- net +5V: no longer U4.10 (IO), U4.16 (VCC), U5.16 (VCC)
Changed lines of the file:
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@@
       (effects (font (size 1.27 1.27)) (justify left))
     )
-    (property "Footprint" "Capacitor_SMD:C_0603_1608Metric_Pad1.08x0.95mm_HandSolder" (id 2) (at 61.9252 54.61 0)
+    (property "Footprint" "Capacitor_THT:CP_Radial_D5.0mm_P2.00mm" (id 2) (at 61.9252 54.61 0)
       (effects (font (size 1.27 1.27)) hide)
     )
@@
       (effects (font (size 1.27 1.27)) (justify left))
     )
-    (property "Footprint" "Capacitor_SMD:C_0603_1608Metric_Pad1.08x0.95mm_HandSolder" (id 2) (at 107.6452 54.61 0)
+    (property "Footprint" "Capacitor_THT:CP_Radial_D5.0mm_P2.00mm" (id 2) (at 107.6452 54.61 0)
       (effects (font (size 1.27 1.27)) hide)
     )
@@
     (pin "1")
     (pin "2")
-  )
-  (symbol (lib_id "power:+5V") (at 176.53 114.3 0) (unit 1)
-    (in_bom yes) (on_board yes) (fields_autoplaced)
-    (property "Reference" "#PWR0102" (id 0) (at 176.53 118.11 0)
-      (effects (font (size 1.27 1.27)) hide)
-    )
-    (property "Value" "+5V" (id 1) (at 176.53 110.7242 0))
-    (property "Footprint" "" (id 2) (at 176.53 114.3 0)
-      (effects (font (size 1.27 1.27)) hide)
-    )
-    (property "Datasheet" "" (id 3) (at 176.53 114.3 0)
-      (effects (font (size 1.27 1.27)) hide)
-    )
-    (pin "1")
   )
   (symbol (lib_id "power:GND") (at 457.2 137.16 0) (unit 1)
@@
     (pin "2")
   )
+  (symbol (lib_id "power:+3V3") (at 176.53 114.3 0) (unit 1)
+    (in_bom yes) (on_board yes) (fields_autoplaced)
+    (property "Reference" "#PWR?" (id 0) (at 176.53 118.11 0)
+      (effects (font (size 1.27 1.27)) hide)
+    )
+    (property "Value" "+3V3" (id 1) (at 176.53 110.7242 0))
+    (property "Footprint" "" (id 2) (at 176.53 114.3 0)
+      (effects (font (size 1.27 1.27)) hide)
+    )
+    (property "Datasheet" "" (id 3) (at 176.53 114.3 0)
+      (effects (font (size 1.27 1.27)) hide)
+    )
+    (pin "1")
+  )
   (symbol (lib_id "Switch:SW_Push") (at 346.71 242.57 0) (unit 1)
     (in_bom yes) (on_board yes)
@@
       (effects (font (size 1.27 1.27)) (justify left))
     )
-    (property "Footprint" "Capacitor_SMD:C_0603_1608Metric_Pad1.08x0.95mm_HandSolder" (id 2) (at 59.9948 73.66 0)
+    (property "Footprint" "Capacitor_THT:CP_Radial_D5.0mm_P2.00mm" (id 2) (at 59.9948 73.66 0)
       (effects (font (size 1.27 1.27)) hide)
     )
@@
       (reference "#PWR0101") (unit 1) (value "+36V") (footprint "")
     )
-    (path "/88c8f5ea-5660-45c6-88ca-6439f84c2291"
-      (reference "#PWR0102") (unit 1) (value "+5V") (footprint "")
-    )
     (path "/d633161c-970e-4fc0-936a-5ca4c8c5cb05"
       (reference "#PWR0103") (unit 1) (value "+5VA") (footprint "")
@@
       (reference "#PWR0106") (unit 1) (value "+5VA") (footprint "")
     )
+    (path "/f5d98a9f-eb8b-481d-b9aa-eb4be56d35b9"
+      (reference "#PWR?") (unit 1) (value "+3V3") (footprint "")
+    )
     (path "/3eb41d07-09c4-4dfd-8b8d-ce489c95f93b"
-      (reference "C1") (unit 1) (value "22uF") (footprint "Capacitor_SMD:C_0603_1608Metric_Pad1.08x0.95mm_HandSolder")
+      (reference "C1") (unit 1) (value "22uF") (footprint "Capacitor_THT:CP_Radial_D5.0mm_P2.00mm")
     )
     (path "/3b98aea0-358a-44d9-8545-7e34dc581b8f"
@@
     )
     (path "/70a4b715-6b96-4b1e-a90b-271ad9d8e6d8"
-      (reference "C4") (unit 1) (value "10uF") (footprint "Capacitor_SMD:C_0603_1608Metric_Pad1.08x0.95mm_HandSolder")
+      (reference "C4") (unit 1) (value "10uF") (footprint "Capacitor_THT:CP_Radial_D5.0mm_P2.00mm")
     )
     (path "/30c80fca-5a9e-4083-a368-28925bfcbf41"
@@
     )
     (path "/fac3f06f-873b-4b1d-a1af-337272363ffa"
-      (reference "C6") (unit 1) (value "22uF") (footprint "Capacitor_SMD:C_0603_1608Metric_Pad1.08x0.95mm_HandSolder")
+      (reference "C6") (unit 1) (value "22uF") (footprint "Capacitor_THT:CP_Radial_D5.0mm_P2.00mm")
     )
     (path "/c6d47a19-ec5e-48d4-af40-72758e09961d"

Commit message: PCB Layout Core Board
Finished
Parts:
- C4: footprint Capacitor_THT:CP_Radial_D5.0mm_P2.00mm -> Capacitor_SMD:C_0603_1608Metric_Pad1.08x0.95mm_HandSolder
Changed lines of the file:
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@@
       (effects (font (size 1.27 1.27)) (justify left))
     )
-    (property "Footprint" "Capacitor_THT:CP_Radial_D5.0mm_P2.00mm" (id 2) (at 107.6452 54.61 0)
+    (property "Footprint" "Capacitor_SMD:C_0603_1608Metric_Pad1.08x0.95mm_HandSolder" (id 2) (at 107.6452 54.61 0)
       (effects (font (size 1.27 1.27)) hide)
     )
@@
   (symbol (lib_id "power:+3V3") (at 176.53 114.3 0) (unit 1)
     (in_bom yes) (on_board yes) (fields_autoplaced)
-    (property "Reference" "#PWR?" (id 0) (at 176.53 118.11 0)
+    (property "Reference" "#PWR0102" (id 0) (at 176.53 118.11 0)
       (effects (font (size 1.27 1.27)) hide)
     )
@@
       (reference "#PWR0101") (unit 1) (value "+36V") (footprint "")
     )
+    (path "/f5d98a9f-eb8b-481d-b9aa-eb4be56d35b9"
+      (reference "#PWR0102") (unit 1) (value "+3V3") (footprint "")
+    )
     (path "/d633161c-970e-4fc0-936a-5ca4c8c5cb05"
       (reference "#PWR0103") (unit 1) (value "+5VA") (footprint "")
@@
       (reference "#PWR0106") (unit 1) (value "+5VA") (footprint "")
     )
-    (path "/f5d98a9f-eb8b-481d-b9aa-eb4be56d35b9"
-      (reference "#PWR?") (unit 1) (value "+3V3") (footprint "")
-    )
     (path "/3eb41d07-09c4-4dfd-8b8d-ce489c95f93b"
       (reference "C1") (unit 1) (value "22uF") (footprint "Capacitor_THT:CP_Radial_D5.0mm_P2.00mm")
@@
     )
     (path "/70a4b715-6b96-4b1e-a90b-271ad9d8e6d8"
-      (reference "C4") (unit 1) (value "10uF") (footprint "Capacitor_THT:CP_Radial_D5.0mm_P2.00mm")
+      (reference "C4") (unit 1) (value "10uF") (footprint "Capacitor_SMD:C_0603_1608Metric_Pad1.08x0.95mm_HandSolder")
     )
     (path "/30c80fca-5a9e-4083-a368-28925bfcbf41"

Commit message: Corrected Capacitor
Parts:
- C4: footprint Capacitor_SMD:C_0603_1608Metric_Pad1.08x0.95mm_HandSolder -> Capacitor_SMD:C_1210_3225Metric_Pad1.33x2.70mm_HandSolder
Changed lines of the file:
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@@
       (effects (font (size 1.27 1.27)) (justify left))
     )
-    (property "Footprint" "Capacitor_SMD:C_0603_1608Metric_Pad1.08x0.95mm_HandSolder" (id 2) (at 107.6452 54.61 0)
+    (property "Footprint" "Capacitor_SMD:C_1210_3225Metric_Pad1.33x2.70mm_HandSolder" (id 2) (at 107.6452 54.61 0)
       (effects (font (size 1.27 1.27)) hide)
     )
@@
     )
     (path "/70a4b715-6b96-4b1e-a90b-271ad9d8e6d8"
-      (reference "C4") (unit 1) (value "10uF") (footprint "Capacitor_SMD:C_0603_1608Metric_Pad1.08x0.95mm_HandSolder")
+      (reference "C4") (unit 1) (value "10uF") (footprint "Capacitor_SMD:C_1210_3225Metric_Pad1.33x2.70mm_HandSolder")
     )
     (path "/30c80fca-5a9e-4083-a368-28925bfcbf41"
