File: Hardware/CoreBoard_Rev1/DriveBoard_Rev2.kicad_sch (KiCad schematic)
At the start: 137 parts, among them J1 RJ45_LED_Shielded, Q1 Q_NMOS_DGS, Q2 Q_NMOS_DGS, Q3 Q_NMOS_DGS, Q4 Q_NMOS_DGS, Q5 Q_NMOS_DGS, Q6 Q_NMOS_DGS, Q7 Q_NMOS_DGS, Q8 Q_NMOS_DGS, Q9 Q_NMOS_DGS, SW1 SW_Push, SW10 SW_Push, SW11 SW_Push, SW12 SW_Push, SW13 SW_Push, SW14 SW_Push, SW15 SW_Push, SW16 SW_SPDT, SW2 SW_Push, SW3 SW_Push, SW4 SW_Push, SW5 SW_Push, SW6 SW_Push, SW7 SW_Push, SW8 SW_Push, SW9 SW_Push, U1 Teensy4.1_DEV-16771, U2 TSR_1-2450, U3 OKI, U4 74HC148, U5 74HC148, U6 74HC00, U7 TSR_1-2450

Commit message: Fixed CoreBoard PCB
Fixed Pin Assignments
Connections:
- net +36V: now also C6.1; no longer C6.2
- net BLRX: now also Conn3.3, U1.0 (RX1); no longer Conn3.9, U1.16 (A2)
- net BLTX: now also Conn3.2, U1.1 (TX1); no longer Conn3.8, U1.17 (A3)
- net FLRX: now also Conn3.9, U1.16 (A2); no longer Conn3.3, U1.0 (RX1)
- net FLTX: now also Conn3.8, U1.17 (A3); no longer Conn3.2, U1.1 (TX1)
- net GND: now also C6.2; no longer C6.1
- net ServoPWM7: now also Conn7.3, U1.12 (MISO); no longer Conn7.9, U1.18 (A4)
- net ServoPWM9: now also Conn7.9, U1.18 (A4); no longer Conn7.3, U1.12 (MISO)
Other:
- moved on the sheet: C6
