File: Hardware/CoreBoard_Rev1/DriveBoard_Rev2.kicad_pcb (KiCad board)
At the start: 2 copper layers, 152.4 x 101.6 mm, 139 parts, among them J1 RJ45_LED_Shielded, Q1 Q_NMOS_DGS, Q2 Q_NMOS_DGS, Q3 Q_NMOS_DGS, Q4 Q_NMOS_DGS, Q5 Q_NMOS_DGS, Q6 Q_NMOS_DGS, Q7 Q_NMOS_DGS, Q8 Q_NMOS_DGS, Q9 Q_NMOS_DGS, SW1 SW_Push, SW10 SW_Push, SW11 SW_Push, SW12 SW_Push, SW13 SW_Push, SW14 SW_Push, SW15 SW_Push, SW16 SW_SPDT, SW2 SW_Push, SW3 SW_Push, SW4 SW_Push, SW5 SW_Push, SW6 SW_Push, SW7 SW_Push, SW8 SW_Push, SW9 SW_Push, U1 Teensy4.1_DEV-16771, U2 TSR_1-2450, U3 OKI, U4 74HC148, U5 74HC148, U6 74HC00, U7 TSR_1-2450

Commit message: Fixed PCB
Parts:
- moved C6 1.91 mm to (75.6, 67.1), turned to 180 degrees
Connections:
- C6 pad 1: GND -> +36V
- C6 pad 2: +36V -> GND
- Conn3 pad 2: FLTX -> BLTX
- Conn3 pad 3: FLRX -> BLRX
- Conn3 pad 8: BLTX -> FLTX
- Conn3 pad 9: BLRX -> FLRX
- Conn7 pad 3: ServoPWM9 -> ServoPWM7
- Conn7 pad 9: ServoPWM7 -> ServoPWM9
- U1 pad 0: FLRX -> BLRX
- U1 pad 1: FLTX -> BLTX
- U1 pad 12: ServoPWM9 -> ServoPWM7
- U1 pad 16: BLRX -> FLRX
- U1 pad 17: BLTX -> FLTX
- U1 pad 18: ServoPWM7 -> ServoPWM9
Routing:
- net FLRX: track 121.4 -> 91.7 mm
- net BLRX: track 91.7 -> 121.4 mm
- net FLTX: track 118.6 -> 91.3 mm
- net BLTX: track 91.3 -> 118.6 mm
- net ServoPWM9: track 170.3 -> 163.3 mm, vias 3 -> 2
- net ServoPWM7: track 163.3 -> 170.3 mm, vias 2 -> 3
