File: drive_board/drive_board.kicad_sch (KiCad schematic)
At the start: 0 parts

Commit message: Hierarchy Sheets
Put empty shit
Parts:
- added H1, H2, H3, H4: MountingHole, MRDT_Shields:RoveNode_H5, symbol Mechanical:MountingHole
- added U1: (no value), MRDT_Shields:RoveNode_H5, symbol MRDT_Shields:RoveNode_H5
Other:
- added sheet Connectors (Connectors.kicad_sch)
- added sheet Motor Controllers (Motor_Controllers.kicad_sch)
- added sheet Power (Power.kicad_sch)
- added sheet Test Buttons (Test_Buttons.kicad_sch)

Commit message: Ethernet ish and Megafit
Parts:
- added C1: C, symbol Device:C
- added J2: RJ45_LED_Shielded, Connector_RJ:RJ45_Wuerth_74980111211_Horizontal, symbol Connector:RJ45_LED_Shielded
Connections:
- new net: C1.1, J2.2
- new net GND: C1.2, J2.8, J2.9, J2.SH
- no-connect marks 0 -> 3
