File: drive_board/drive_board.kicad_sch (KiCad schematic)
At the start: 20 parts, among them J10 Conn_01x02_Pin, J11 Conn_01x04_Pin, J2 RJ45_LED_Shielded, J3 Conn_01x02_Pin, J4 Conn_01x02_Pin, J5 Conn_01x02_Pin, J6 Conn_01x02_Pin, J7 Conn_01x02_Pin, J8 Conn_01x02_Pin, J9 Conn_01x02_Pin, U2 SN65HVD232

Commit message: Finish Schematic
- Assigned all footprints
- Added dipswitch and connected to RoveNode
- Updated PCB from schematic
- Added absolute encoder pins and connected to RoveNode
Parts:
- added J11, J12, J13, J14: Conn_01x03_Pin, Connector_JST:JST_PH_B3B-PH-K_1x03_P2.00mm_Vertical, symbol Connector:Conn_01x03_Pin
- C1, C3, C4: footprint (none) -> Capacitor_SMD:C_0603_1608Metric_Pad1.08x0.95mm_HandSolder
- H1, H2, H3, H4: footprint (none) -> MRDT_Drill_Holes:4_40_Hole_Pad_Via
- J10, J3, J4, J5, J6, J7, J8, J9: footprint Package_DFN_QFN:QFN-20-1EP_5x5mm_P0.65mm_EP3.35x3.35mm -> Connector_JST:JST_PH_B2B-PH-K_1x02_P2.00mm_Vertical
- J15: renamed from J11; footprint Package_DIP:DIP-20_W7.62mm -> Connector_JST:JST_PH_B4B-PH-K_1x04_P2.00mm_Vertical
Connections:
- net +3.3V is gone; now on net +3V3: U1.3 (3V3)
- net Back_Input is gone; now on net JYSTK1_HORIZ: U1.43 (PB1)
- net Forward_Input is gone; now on net JYSTK1_VERT: U1.42 (PB0)
- net Left_Input is gone; now on net JYSTK1_PRS: U1.44 (PB2)
- net +3V3: now also J11.3 (Pin_3), J12.3 (Pin_3), J13.3 (Pin_3), J14.3 (Pin_3)
- net GND: now also J11.2 (Pin_2), J12.2 (Pin_2), J13.2 (Pin_2), J14.2 (Pin_2)
- net JYSTK1_HORIZ: no longer U1.11 (PA9)
- net JYSTK1_PRS: no longer U1.12 (PA8)
- net JYSTK1_VERT: no longer U1.10 (PA10)
- net JYSTK2_HORIZ: now also U1.11 (PA9); no longer U1.40 (PA4)
- net JYSTK2_PRS: now also U1.10 (PA10); no longer U1.41 (PA6)
- net JYSTK2_VERT: now also U1.12 (PA8); no longer U1.39 (PA3)
- net UART4_TX: now also U1.8 (PC10); no longer U1.38 (PA0)
- net FNT_RGHT_ABS_ENC: now reaches U1.17 (PB14)
- net FNT_RGHT_ABS_ENC: now also J12.1 (Pin_1)
- net FNT_LFT_TURN_SW: now reaches U1.25 (PD2)
- net FNT_LFT_WHL_SW: now reaches U1.26 (PB4)
- net FNT_RGHT_TURN_SW: now reaches U1.36 (PC2)
- net FNT_RGHT_WHL_SW: now reaches U1.37 (PC3)
- net BCK_LFT_ABS_ENC: now reaches U1.6 (PC12)
- net BCK_LFT_ABS_ENC: now also J13.1 (Pin_1)
- net FNT_LFT_ABS_ENC: now reaches U1.9 (PA15)
- net FNT_LFT_ABS_ENC: now also J11.1 (Pin_1)
- net BCK_LFT_TURN_MOT renamed BCK_LFT_TURN_LED
- net BCK_LFT_WHL_MOT renamed BCK_LFT_WHL_LED
- net BCK_RGHT_TURN_MOT renamed BCK_RGHT_TURN_LED
- net BCK_RGHT_WHL_MOT renamed BCK_RGHT_WHL_LED
- net FNT_LFT_TURN_MOT renamed FNT_LFT_TURN_LED
- net FNT_LFT_WHL_MOT renamed FNT_LFT_WHL_LED
- net FNT_RGHT_TURN_MOT renamed FNT_RGHT_TURN_LED
- net FNT_RGHT_WHL_MOT renamed FNT_RGHT_WHL_LED
- net Right_Input renamed BCK_RGHT_WHL_SW
- new net BCK_LFT_TURN_SW: U1.39 (PA3)
- new net BCK_LFT_WHL_SW: U1.40 (PA4)
- new net BCK_RGHT_ABS_ENC: J14.1 (Pin_1), U1.38 (PA0)
- new net BCK_RGHT_TURN_SW: U1.41 (PA6)
- no-connect marks 9 -> 1
Other:
- sheet Test Buttons ports: added BCK_LFT_TURN_LED, BCK_LFT_TURN_SW, BCK_LFT_WHL_LED, BCK_LFT_WHL_SW, BCK_RGHT_TURN_LED, BCK_RGHT_TURN_SW, BCK_RGHT_WHL_LED, BCK_RGHT_WHL_SW, FNT_LFT_TURN_LED, FNT_LFT_TURN_SW, FNT_LFT_WHL_LED, FNT_LFT_WHL_SW, FNT_RGHT_TURN_LED, FNT_RGHT_TURN_SW, FNT_RGHT_WHL_LED, FNT_RGHT_WHL_SW; removed BLMOT_T, BLMOT_W, BRMOT_T, BRMOT_W, FLMOT_T, FLMOT_W, FRMOT_T, FRMOT_W
- note added: "<- (just in case.)"
- moved on the sheet: J10, J15, J3, J4, J5, J6, J7, J8, J9

Commit message: Finish first draft
B approved
Did everything
Made room for traces
Placed everything in places
Parts:
- J2: footprint Connector_RJ:RJ45_Wuerth_74980111211_Horizontal -> MRDT_Connectors:RJ45_Teensy
Changed lines of the file:
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@@
 			)
 		)
-		(property "Footprint" "Connector_RJ:RJ45_Wuerth_74980111211_Horizontal"
+		(property "Footprint" "MRDT_Connectors:RJ45_Teensy"
 			(at 56.515 157.48 90)
 			(hide yes)
