File: drive_board/drive_board.kicad_pcb (KiCad board)
At the start: 2 copper layers, 77 parts, among them J1 Molex_Megafit_02, J10 Conn_01x02_Pin, J11 Conn_01x03_Pin, J12 Conn_01x03_Pin, J13 Conn_01x03_Pin, J14 Conn_01x03_Pin, J15 Conn_01x04_Pin, J2 RJ45_LED_Shielded, J3 Conn_01x02_Pin, J4 Conn_01x02_Pin, J5 Conn_01x02_Pin, J6 Conn_01x02_Pin, J7 Conn_01x02_Pin, J8 Conn_01x02_Pin, J9 Conn_01x02_Pin, Q12 BSS138, Q13 BSS138, Q14 BSS138, Q15 BSS138, Q16 BSS138, Q17 BSS138, Q18 BSS138, Q19 BSS138, U2 SN65HVD232, U3 COM-09032, U4 COM-09032, U5 4-1825059-2

Commit message: pcb layout orginization
placed most components in respective areas on the board
(fixed a bit of the mess)
Parts:
- moved J2 164.5 mm to (159.1, 144.5)
- moved H2 164.1 mm to (152.5, 122.4)
- moved J15 159.8 mm to (175.5, 81.5), turned to 180 degrees
- moved J8 154.5 mm to (175.4, 128.0), turned to 90 degrees
- moved J7 152.8 mm to (168.1, 128.0), turned to 90 degrees
- moved H1 150.7 mm to (168.3, 67.1)
- moved J10 143.9 mm to (175.4, 120.4), turned to 90 degrees
- moved C1 143.0 mm to (154.4, 131.8)
- moved J9 142.1 mm to (168.1, 120.4), turned to 90 degrees
- moved J3 138.9 mm to (163.1, 80.0), turned to -90 degrees
- moved J5 138.8 mm to (160.3, 102.9), turned to 180 degrees
- moved U1 134.3 mm to (114.8, 70.3)
- moved J6 132.2 mm to (160.3, 95.5), turned to 180 degrees
- moved U2 131.8 mm to (158.9, 111.8), turned to 90 degrees
- moved R24 131.0 mm to (159.2, 90.2)
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
Commit message: Finish first draft
B approved
Did everything
Made room for traces
Placed everything in places
Parts:
- J1: footprint MRDT_Connectors:MOLEX_MegaFit_02_Horizontal -> megafit:CONN_SD-768290002_02_MOL
- J2: footprint Connector_RJ:RJ45_Wuerth_74980111211_Horizontal -> MRDT_Connectors:RJ45_Teensy
- moved H3 226.6 mm to (243.8, 99.1), turned to 90 degrees
- moved U4 186.1 mm to (197.6, 92.5), turned to -90 degrees
- moved C3 158.5 mm to (188.3, 60.3), turned to -90 degrees
- moved U3 158.3 mm to (169.0, 92.6), turned to -90 degrees
- moved C4 156.1 mm to (185.8, 60.3), turned to -90 degrees
- moved D17 152.3 mm to (234.4, 95.5)
- moved D12 152.2 mm to (234.3, 84.8), turned to 180 degrees
- moved D14 152.1 mm to (234.6, 98.8)
- moved D10 151.9 mm to (234.3, 87.6), turned to 180 degrees
- moved R26 150.7 mm to (241.1, 64.1), turned to 90 degrees
- moved J12 149.6 mm to (195.8, 37.6)
- moved R25 147.7 mm to (238.6, 64.1), turned to 90 degrees
- moved R20 147.0 mm to (231.4, 64.1), turned to 90 degrees
- moved Q15 145.8 mm to (236.1, 70.6)
- moved R22 144.6 mm to (236.1, 64.1), turned to 90 degrees
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Connections:
- U5 pad 1: +3.3V -> +3V3
- U5 pad 2: +3.3V -> +3V3
- U5 pad 3: +3.3V -> +3V3
- U5 pad 4: +3.3V -> +3V3
- U5 pad 5: +3.3V -> +3V3
- U5 pad 6: +3.3V -> +3V3
- U5 pad 7: +3.3V -> +3V3
- U5 pad 8: +3.3V -> +3V3
Other:
- board outline added: 121.9 x 78.7 mm
